File: Demo/Egret.kicad_sch (KiCad schematic)
At the start: 6 parts

Commit message: update
Parts:
- added C? (x3): C, symbol Device:C
- gave numbers to parts that had none: 6
Connections:
- net at U2.2 (GND): now also C?.2
- net at U2.5 (VOUT): now also C?.2, C?.2
- new net GND: C?.1, C?.1, C?.1

Commit message: update
Parts:
- added Q? (x2): S8050, Package_TO_SOT_THT:TO-92_Inline, symbol Transistor_BJT:S8050
- added R? (x4): R, symbol Device:R
- gave numbers to parts that had none: 3
Connections:
- net +5V: now also U2.1 (VIN), U2.4 (BYPASS), U4.7 (VREGIN), U4.8 (VBUS), R?.1
- net GND: now also U2.3 (ON/~{OFF}), U4.29 (GND), U4.3 (GND)
- net +3.3V: now reaches C1.2, C3.2, U2.5 (VOUT)
- net RTS: now reaches U4.24 (RTS)
- net RTS: now also Q?.3 (C), R?.2
- net CP_Rx: now reaches U4.25 (RXD)
- net at U4.26 (TXD): now also R?.2
- net DTR: now reaches U4.28 (DTR)
- net DTR: now also Q?.1 (E), R?.2
- net USB-PWR-DM: now reaches U4.4 (D+)
- net USB-PWR-DP: now reaches U4.5 (D-)
- net at U4.9 (~{RST}): now also R?.2
- new net: Q?.2 (B), R?.1 (x2)
- new net CP_Tx: R?.1
- new net EN: Q?.1 (E)
- new net GPIO0: Q?.3 (C)
- no-connect marks 0 -> 18
Other:
- moved on the sheet: C1, C2, C3, J1, U1, U2, U3, U4, U5

Commit message: update
Parts:
- added C? (x5): C, symbol Device:C
- added J?: 2388749-1, TE_2388749-1, symbol 2388749-1:2388749-1
- added R? (x2): R, symbol Device:R
- added U?: AN2051, AN2051, symbol AN2051:AN2051
- gave numbers to parts that had none: 6
Connections:
- net +3.3V: now also R?.1; no longer C1.2, C3.2, U2.5 (VOUT)
- net +5V: now also J?.A4 (VBUS_A), J?.A9 (VBUS_A)
- net CP_Rx: now also U5.41 (U0TXD)
- net CP_Tx: now also U5.40 (U0RXD)
- net GND: now also U1.1 (CLKIN), U1.11 (FYSNC), U1.9 (AD0), U5.49 (GND), C?.2, C?.2, C?.2, C?.2, J?.A1 (GND_A), J?.A12 (GND_A), J?.B1 (GND_B), J?.B12 (GND_B), J?.S1 (SHIELD), J?.S2 (SHIELD), J?.S3 (SHIELD), J?.S4 (SHIELD)
- net GPIO0: now also U5.23 (IO0)
- net USB-PWR-DM: now also J?.A7 (DN1), J?.B7 (DN2)
- net USB-PWR-DP: now also J?.A6 (DP1), J?.B6 (DP2)
- net at U1.10 (REGOUT): now also C?.1
- net +3V3: now reaches U1.13 (VDD)
- net +3V3: now also C1.2, C3.2, U2.5 (VOUT), C?.1
- net MPU_SCL: now reaches U1.23 (SCL)
- net MPU_SDA: now reaches U1.24 (SDA)
- net 3V3A: now reaches U5.1 (VDDA), U5.43 (VDDA), U5.46 (VDDA)
- net 3V3A: now also U5.19 (VDD3P3_RTC), U5.3 (VDDA3P3), U5.37 (VDD3P3_CPU), U5.4 (VDDA3P3), C?.1, C?.1, R?.2
- net GPIO34: now reaches U5.10 (IO34)
- net GPIO35: now reaches U5.11 (IO35)
- net GPIO32: now reaches U5.12 (IO32)
- net GPIO33: now reaches U5.13 (IO33)
- net GPIO25: now reaches U5.14 (IO25)
- net GPIO26: now reaches U5.15 (IO26)
- net GPIO27: now reaches U5.16 (IO27)
- net GPIO14: now reaches U5.17 (IO14)
- net GPIO12: now reaches U5.18 (IO12)
- net at U5.2 (LNA_IN): now also U?.P$1 (FEED), U?.P$2 (SODLER)
- net GPIO13: now reaches U5.20 (IO13)
- net GPIO15: now reaches U5.21 (IO15)
- net GPIO2: now reaches U5.22 (IO2)
- net GPIO4: now reaches U5.24 (IO4)
- net FLASH_CS: now reaches U5.25 (IO16)
- net FLASH_SD0: now reaches U5.27 (IO17)
- net GPIO9: now reaches U5.28 (SD2)
- net GPIO10: now reaches U5.29 (SD3)
- net FLASH_SD2: now reaches U5.30 (CMD)
- net FLASH_CLK: now reaches U5.31 (CLK)
- net FLASH_SD3: now reaches U5.32 (SD0)
- net FLASH_SD1: now reaches U5.33 (SD1)
- net GPIO5: now reaches U5.34 (IO5)
- net GPIO18: now reaches U5.35 (IO18)
- net GPIO23: now reaches U5.36 (IO23)
- net GPIO19: now reaches U5.38 (IO19)
- net GPIO22: now reaches U5.39 (IO22)
- net GPIO21: now reaches U5.42 (IO21)
- net SENSOR_VP: now reaches U5.5 (SENSOR_VP)
- net GPIO37: now reaches U5.6 (SENSOR_CAPP)
- net GPIO38: now reaches U5.7 (SENSOR_CAPN)
- net SENSOR_VN: now reaches U5.8 (SENSOR_VN)
- net CHIP_PU: now reaches U5.9 (EN)
- new net: J?.B4 (VBUS_B), J?.B9 (VBUS_B)
- no-connect marks 18 -> 30
Other:
- moved on the sheet: C1, C2, C3, J1, Q1, Q2, R1, R2, R3, R4, U1, U2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

Commit message: update
Parts:
- removed C?: C, symbol Device:C
- removed R?: R, symbol Device:R
- added C?: 2.2nF, symbol Device:C
- added C?: 10nF, symbol Device:C
- C?: value C -> 0.1uF
Connections:
- net +3.3V is gone; now on net +3V3: R?.1
- net +3V3: now also U1.8 (VLOGIC), C?.1
- net GND: now also U1.18 (GND), C?.2, C?.2
- net at U1.20 (CPOUT): now also C?.1
- no-connect marks 30 -> 35
Other:
- moved on the sheet: C?, J1, R?, U1, U3, U5, U?

Commit message: update
Parts:
- added R? (x4): R, symbol Device:R
Connections:
- net +3V3: now also J1.4 (VDD), R?.2, R?.2, R?.2, R?.2
- net GND: now also J1.6 (VSS), J1.9 (SHIELD)
- net SD_CS: now reaches J1.2 (DAT3/CD)
- net SD_CS: now also R?.1
- net SD_MOS: now reaches J1.3 (CMD)
- net SD_CLK: now reaches J1.5 (CLK)
- net SD_CLK: now also R?.1
- net SD_MISO: now reaches J1.7 (DAT0)
- net SD_MISO: now also R?.1
- new net SD_MOSI: R?.1
- no-connect marks 35 -> 37
Other:
- moved on the sheet: C?, J1, R?, U1, U3, U5, U?

Commit message: update
Parts:
- gave numbers to parts that had none: 13

Commit message: update
Parts:
- added C8: 0.1uF, symbol Device:C
- added J1: Conn_01x08_Male, symbol Connector:Conn_01x08_Male
- added R1: 10k, symbol Device:R
- C10: renamed from C9; value C -> 10uF
- C2: renamed from C4; value C -> 0.1uF
- C5: renamed from C1; value C -> 0.1uF
- C6: renamed from C3; value C -> 10uF
- C9: renamed from C8; value C -> 0.1uF
- R2: renamed from R3; value R -> 12k
- R3: renamed from R4; value R -> 12k
- R4: renamed from R1; value R -> 200R
- R5: renamed from R2; value R -> 10k
- R6: renamed from R5; value R -> 0
- renumbered C2 to C1, C5 to C3, C6 to C4, J1 to J2, J2 to J3, R9 to R10, R6 to R7, R7 to R8, R8 to R9, U5 to U4, U6 to U5, U4 to U6
Connections:
- net CHIP_PU is gone; now on net EN: U4.9 (EN)
- net MPU_SCL is gone; now on net BH_SCL: U1.23 (SCL)
- net MPU_SDA is gone; now on net BH_SDA: U1.24 (SDA)
- net SD_CLK is gone; now on net GPIO14: J2.5 (CLK), R9.1
- net SD_CS is gone; now on net GPIO15: J2.2 (DAT3/CD), R10.1
- net SD_MISO is gone; now on net GPIO26: J2.7 (DAT0), R7.1
- net SD_MOS is gone; now on net GPIO13: J2.3 (CMD)
- net SD_MOSI is gone; now on net GPIO13: R8.1
- net +3V3: now also J1.7 (Pin_7), R1.1
- net +5V: now also J3.B4 (VBUS_B), J3.B9 (VBUS_B), U2.3 (ON/~{OFF}), U3.1 (VDD), J1.8 (Pin_8); no longer U2.4 (BYPASS)
- net EN: now also Q1.3 (C), C8.1, R1.2; no longer Q1.1 (E)
- net GND: now also C1.2, U2.2 (GND), U3.3 (VSS), C8.2, J1.6 (Pin_6); no longer C1.1, U2.3 (ON/~{OFF})
- net GPIO18: now also J1.4 (Pin_4)
- net GPIO23: now also J1.3 (Pin_3)
- net GPIO27: now also U3.4 (DIN)
- net GPIO4: now also J1.2 (Pin_2)
- net GPIO5: now also J1.1 (Pin_1)
- net RTS: now also Q1.1 (E); no longer Q1.3 (C)
- net USB-PWR-DM: now also U6.5 (D-); no longer U6.4 (D+)
- net USB-PWR-DP: now also U6.4 (D+); no longer U6.5 (D-)
- net at U4.2 (LNA_IN), U5.P$2 (SODLER): no longer U5.P$1 (FEED)
- net GPIO2 renamed DC
- net DC: now also J1.5 (Pin_5)
- net GPIO32 renamed BH_SDA
- net GPIO33 renamed BH_SCL
- new net: C1.1, U2.4 (BYPASS)
- no-connect marks 37 -> 40
Other:
- note added: "GPIO"
- note added: "TF 存储卡"
- note added: "USB 转串口芯片"
- note added: "加速度传感器"
- note added: "微控制器"
- note added: "扩展板"
- note added: "线性稳压器"
- moved on the sheet: C1, C10, C2, C3, C4, C5, C6, C7, C9, J2, J3, Q1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
