File: Demo/Egret.kicad_sch (KiCad schematic)
At the start: 31 parts, among them J1 Conn_01x08_Male, J2 Micro_SD_Card, J3 2388749-1, Q1 S8050, Q2 S8050, U1 MPU6050, U2 LP2992IM5-3.3, U3 WS2812B-B, U4 ESP32-PICO-D4, U5 AN2051, U6 CP2102N-A01-GQFN28

Commit message: update
Parts:
- added C5: 0.1uF, Capacitor_SMD:C_0603_1608Metric, symbol Device:C
- added R1: 10k, Resistor_SMD:R_0603_1608Metric, symbol Device:R
- added U3: BH1750FVI-TR, BH1750FVI-TR:XDCR_BH1750FVI-TR, symbol BH1750FVI-TR:BH1750FVI-TR
- C1: value C -> 10nF; footprint (none) -> Capacitor_SMD:C_0603_1608Metric
- C10: renamed from C9; footprint (none) -> Capacitor_SMD:C_0603_1608Metric
- C11: renamed from C10; footprint (none) -> Capacitor_SMD:C_0603_1608Metric
- C2, C3, C4: footprint (none) -> Capacitor_SMD:C_0603_1608Metric
- C6: renamed from C5; footprint (none) -> Capacitor_SMD:C_0603_1608Metric
- C7: renamed from C6; footprint (none) -> Capacitor_SMD:C_0603_1608Metric
- C8: renamed from C7; footprint (none) -> Capacitor_SMD:C_0603_1608Metric
- C9: renamed from C8; footprint (none) -> Capacitor_SMD:C_0603_1608Metric
- J1: footprint (none) -> Connector_FFC-FPC:TE_0-1734839-8_1x08-1MP_P0.5mm_Horizontal
- J2: footprint (none) -> Connector_Card:microSD_HC_Molex_104031-0811
- J3: footprint TE_2388749-1 -> 2388749-1:TE_2388749-1
- Q1, Q2: footprint Package_TO_SOT_THT:TO-92_Inline -> Package_TO_SOT_SMD:SOT-23
- R10: renamed from R9; value R -> 10k; footprint (none) -> Resistor_SMD:R_0603_1608Metric
- R11: renamed from R10; value R -> 10k; footprint (none) -> Resistor_SMD:R_0603_1608Metric
- R2: renamed from R1; footprint (none) -> Resistor_SMD:R_0603_1608Metric
- R3: renamed from R2; footprint (none) -> Resistor_SMD:R_0603_1608Metric
- R4: renamed from R3; footprint (none) -> Resistor_SMD:R_0603_1608Metric
- R5: renamed from R4; footprint (none) -> Resistor_SMD:R_0603_1608Metric
- R6: renamed from R5; footprint (none) -> Resistor_SMD:R_0603_1608Metric
- R7: renamed from R6; footprint (none) -> Resistor_SMD:R_0603_1608Metric
- R8: renamed from R7; value R -> 10k; footprint (none) -> Resistor_SMD:R_0603_1608Metric
- R9: renamed from R8; value R -> 10k; footprint (none) -> Resistor_SMD:R_0603_1608Metric
- U1: footprint IC_MPU6050 -> MPU6050:IC_MPU6050
- U2: footprint SOT95P280X145-5N -> LP2992IM5-3:SOT95P280X145-5N
- U4: renamed from U3; footprint LED_WS2812B-B -> WS2812B-B:LED_WS2812B-B
- U5: renamed from U4; footprint PQFN50P700X700X104-49N -> ESP32-PICO-D4:PQFN50P700X700X104-49N
- U6: renamed from U5; footprint AN2051 -> AN2051:AN2051
- U7: renamed from U6; footprint QFN50P500X500X80-29N -> CP2102N-A01-GQFN28:QFN50P500X500X80-29N
Connections:
- net +3V3: now also C5.1, R1.2, U3.1 (VCC)
- net BH_SCL: now also U3.6 (SCL)
- net BH_SDA: now also U3.4 (SDA)
- net GND: now also C5.2, U3.2 (ADDR), U3.3 (GND)
- new net: R1.1, U3.5 (DVI)
Other:
- note added: "扩展板接口"
- note removed: "GPIO"
- note removed: "扩展板"
- moved on the sheet: C2, C3, C4, C8, J1, R10, R8, R9, U1, U4

Commit message: update
Parts:
- removed J3: 2388749-1, 2388749-1:TE_2388749-1, symbol 2388749-1:2388749-1
- added J3: USB_C_Receptacle, Connector_USB:USB_C_Receptacle_XKB_U262-16XN-4BVC11, symbol Connector:USB_C_Receptacle
- renumbered C6 to C5, C7 to C6, C8 to C7, C5 to C8, U4 to U2, U2 to U3, U3 to U4
Connections:
- net +5V: now also J3.A4 (VBUS), J3.A9 (VBUS), J3.B4 (VBUS), J3.B9 (VBUS)
- net GND: now also J3.A1 (GND), J3.A12 (GND), J3.B1 (GND), J3.B12 (GND), J3.S1 (SHIELD)
- net USB-PWR-DM: now also J3.A7 (D-), J3.B7 (D-)
- net USB-PWR-DP: now also J3.A6 (D+), J3.B6 (D+)

Commit message: update
Parts:
- removed C8: 0.1uF, Capacitor_SMD:C_0603_1608Metric, symbol Device:C
- removed J1: Conn_01x08_Male, Connector_FFC-FPC:TE_0-1734839-8_1x08-1MP_P0.5mm_Horizontal, symbol Connector:Conn_01x08_Male
- removed J3: USB_C_Receptacle, Connector_USB:USB_C_Receptacle_XKB_U262-16XN-4BVC11, symbol Connector:USB_C_Receptacle
- removed U6: AN2051, AN2051:AN2051, symbol AN2051:AN2051
- added C9: 0.1uF, Capacitor_SMD:C_0603_1608Metric, symbol Device:C
- added FPC1: FPC-05F-12PH20, kicad_lceda:FPC-SMD_12P-P0.50_FPC-05F-12PH20, symbol kicad_lceda:FPC-05F-12PH20
- added Q3: AO3415AL, kicad_lceda:SOT-23-3_L2.9-W1.6-P1.90-LS2.9-BL, symbol kicad_lceda:AO3415AL
- added R5: 1k, Resistor_SMD:R_0603_1608Metric, symbol Device:R
- added U6: AN2051-245_2.4G全向天线, kicad_lceda:ANT-SMD_L5.0-W2.0, symbol kicad_lceda:AN2051-245_2.4G全向天线
- added USB1: TYPEC-304J-BCP16, kicad_lceda:USB-C-SMD_TYPEC-304J-BCP16, symbol kicad_lceda:TYPEC-304J-BCP16
- J1: renamed from J2; footprint Connector_Card:microSD_HC_Molex_104031-0811 -> Connector_Card:microSD_HC_Wuerth_693072010801
- renumbered C5 to C2, C2 to C3, C3 to C4, C4 to C5, C9 to C8, R9 to R10, R10 to R11, R11 to R12, R5 to R6, R6 to R7, R7 to R8, R8 to R9, U2 to U1, U1 to U2
Connections:
- net +3V3: now also C9.1, FPC1.4, Q3.2 (S)
- net +5V: now also USB1.A4B9 (VBUS)
- net GND: now also C9.2, FPC1.1, FPC1.12, FPC1.2, FPC1.5, FPC1.6, FPC1.8, USB1.13 (GND), USB1.14 (GND), USB1.15 (GND), USB1.16 (GND), USB1.A1B12 (GND)
- net USB-PWR-DM: now also USB1.A7 (DN1), USB1.B7 (DN2)
- net USB-PWR-DP: now also USB1.A6 (DP1), USB1.B6 (DP2)
- net at U5.2 (LNA_IN): now also U6.1 (ANT)
- net BH_SCL renamed GPIO33/MPU_SCL/BH_SCL
- net BH_SDA renamed GPIO32/MPU_SDA/BH_SDA
- net DC renamed GPIO2/DC
- net GPIO2/DC: now also FPC1.7
- net GPIO13 renamed GPIO13/SD_MOSI
- net GPIO14 renamed GPIO14/SD_CLK
- net GPIO15 renamed GPIO15/SD_CS
- net GPIO18 renamed GPIO18/SCK
- net GPIO18/SCK: now also FPC1.9
- net GPIO23 renamed GPIO23/MOSI
- net GPIO26 renamed GPIO26/SD_MISO
- net GPIO26/SD_MISO: now also FPC1.10
- net GPIO27 renamed GPIO27/RGB_LED
- net GPIO34: no longer names the net of U5.10 (IO34)
- net GPIO35: no longer names the net of U5.11 (IO35)
- net GPIO37: no longer names the net of U5.6 (SENSOR_CAPP)
- net GPIO38: no longer names the net of U5.7 (SENSOR_CAPN)
- net GPIO4 renamed GPIO4/RES
- net GPIO4/RES: now also FPC1.11
- net GPIO5 renamed GPIO5/LCD_BL
- net GPIO5/LCD_BL: now also R5.2
- net SENSOR_VN: no longer names the net of U5.8 (SENSOR_VN)
- net SENSOR_VP: no longer names the net of U5.5 (SENSOR_VP)
- new net: Q3.1 (G), R5.1
- new net: FPC1.3, Q3.3 (D)
- no-connect marks 40 -> 41
Other:
- note added: "ST7789 液晶屏"
- note removed: "扩展板接口"
- moved on the sheet: C10, C11, C3, C4, C5, C7, C8, J1, R2, R8, U1, U2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

Commit message: update
Parts:
- removed J1: Micro_SD_Card, Connector_Card:microSD_HC_Wuerth_693072010801, symbol Connector:Micro_SD_Card
- added Card1: TF-02A_C2889261, TF-SMD_TF-02:TF-SMD_TF-02, symbol TF-SMD_TF-02:TF-02A_C2889261
Connections:
- net +3V3: now also Card1.4 (VDD)
- net GND: now also Card1.10 (GND), Card1.11 (GND), Card1.12 (GND), Card1.13 (GND), Card1.6 (VSS), Card1.9 (CD)
- net GPIO13/SD_MOSI: now also Card1.3 (CMD)
- net GPIO14/SD_CLK: now also Card1.5 (CLK)
- net GPIO15/SD_CS: now also Card1.2 (CD/DAT3)
- net GPIO26/SD_MISO: now also Card1.7 (DAT0)
Other:
- moved on the sheet: R10, R11, R12, R9

Commit message: update
Connections:
- net GPIO23/MOSI: now also FPC1.10
- net GPIO26/SD_MISO: no longer FPC1.10
- no-connect marks 41 -> 42
Changed lines of the file:
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@@
   (no_connect (at 194.31 147.32))
   (no_connect (at 194.31 165.1))
+  (no_connect (at 92.456 168.91))
   (no_connect (at 348.742 73.152))
   (no_connect (at 194.31 154.94))
@@
     (effects (font (size 1.27 1.27)) (justify right bottom))
   )
-  (label "GPIO26{slash}SD_MISO" (at 248.412 263.652 180)
-    (effects (font (size 1.27 1.27)) (justify right bottom))
-  )
+  (label "GPIO23{slash}MOSI" (at 248.412 263.652 180)
+    (effects (font (size 1.27 1.27)) (justify right bottom))
+  )

Commit message: update
Connections:
- net USB-PWR-DM renamed USB-PWR-DN
Changed lines of the file:
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@@
     (effects (font (size 1.27 1.27)) (justify left bottom))
   )
-  (label "USB-PWR-DM" (at 348.742 55.372 180)
+  (label "USB-PWR-DN" (at 348.742 55.372 180)
     (effects (font (size 1.27 1.27)) (justify right bottom))
   )
@@
     (effects (font (size 1.27 1.27)) (justify right bottom))
   )
-  (label "USB-PWR-DM" (at 246.38 62.23 180)
+  (label "USB-PWR-DN" (at 246.38 62.23 180)
     (effects (font (size 1.27 1.27)) (justify right bottom))
   )
@@
     (effects (font (size 1.27 1.27)) (justify left bottom))
   )
-  (label "USB-PWR-DM" (at 348.742 70.612 180)
+  (label "USB-PWR-DN" (at 348.742 70.612 180)
     (effects (font (size 1.27 1.27)) (justify right bottom))
   )
