File: Demo/Egret.kicad_pcb (KiCad board)
At the start: 2 copper layers, 43.6 x 33.2 mm, 37 parts, among them Q1 S8050, Q2 S8050, Q3 AO3415AL, U1 WS2812B-B, U2 MPU6050, U3 LP2992IM5-3.3, U4 BH1750FVI-TR, U5 ESP32-PICO-D4, U6 AN2051-245_2.4G全向天线, U7 CP2102N-A01-GQFN28

Commit message: update
Parts:
- moved ? 1.34 mm to (140.6, 97.4)
- moved C4 1.00 mm to (109.3, 90.1)
- moved C5 1.00 mm to (109.3, 83.6)
- moved C7 1.00 mm to (109.3, 85.8)
- moved C3 1.00 mm to (109.3, 88.0)
- moved USB1 0.43 mm to (109.6, 96.8)
Changed lines of the file:
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@@
   )
   (footprint "Capacitor_SMD:C_0603_1608Metric" (layer "F.Cu")
-    (at 109.34 82.5775)
+    (at 109.27 83.58)
     (descr "Capacitor SMD 0603 (1608 Metric), square (rectangular) end terminal, IPC_7351 nominal, (Body size source: IPC-SM-782 page 76, https://www.pcb-3d.com/wordpress/wp-content/uploads/ipc-sm-782a_amendment_1_and_2.pdf), generated with kicad-footprint-generator")
     (tags "capacitor")
@@
   )
   (footprint "Capacitor_SMD:C_0603_1608Metric" (layer "F.Cu")
-    (at 109.359167 86.966834)
+    (at 109.289167 87.969334)
     (descr "Capacitor SMD 0603 (1608 Metric), square (rectangular) end terminal, IPC_7351 nominal, (Body size source: IPC-SM-782 page 76, https://www.pcb-3d.com/wordpress/wp-content/uploads/ipc-sm-782a_amendment_1_and_2.pdf), generated with kicad-footprint-generator")
     (tags "capacitor")
@@
   )
   (footprint "Capacitor_SMD:C_0603_1608Metric" (layer "F.Cu")
-    (at 109.34 84.7775)
+    (at 109.27 85.78)
     (descr "Capacitor SMD 0603 (1608 Metric), square (rectangular) end terminal, IPC_7351 nominal, (Body size source: IPC-SM-782 page 76, https://www.pcb-3d.com/wordpress/wp-content/uploads/ipc-sm-782a_amendment_1_and_2.pdf), generated with kicad-footprint-generator")
     (tags "capacitor")
@@
   )
   (footprint "Capacitor_SMD:C_0603_1608Metric" (layer "F.Cu")
-    (at 109.34 89.1275)
+    (at 109.27 90.13)
     (descr "Capacitor SMD 0603 (1608 Metric), square (rectangular) end terminal, IPC_7351 nominal, (Body size source: IPC-SM-782 page 76, https://www.pcb-3d.com/wordpress/wp-content/uploads/ipc-sm-782a_amendment_1_and_2.pdf), generated with kicad-footprint-generator")
     (tags "capacitor")
@@
   )
   (footprint "kicad_lceda:USB-C-SMD_TYPEC-304J-BCP16" (layer "F.Cu")
-    (at 109.596 96.35 -90)
+    (at 109.59 96.78 -90)
     (property "Sheetfile" "Egret.kicad_sch")
     (property "Sheetname" "")
@@
   )
   (footprint "G+D:logo" (layer "B.Cu")
-    (at 139.29658 97.304102 -90)
+    (at 140.63658 97.354102 -90)
     (attr board_only exclude_from_pos_files exclude_from_bom)
     (fp_text reference "" (at 0 0 90) (layer "B.SilkS")
@@
   )
   (via (at 140.68 88.44) (size 5) (drill 3) (layers "F.Cu" "B.Cu") (free) (net 0))
-  (via (at 140.675 106.325) (size 5) (drill 3) (layers "F.Cu" "B.Cu") (free) (net 0))
+  (via (at 140.76 106.32) (size 5) (drill 3) (layers "F.Cu" "B.Cu") (free) (net 0))
 )

Commit message: update
Parts:
- moved U3 1.01 mm to (110.3, 105.3)
- moved USB1 0.68 mm to (109.5, 97.5)
Connections:
- FPC1 pad 10: /GPIO26/SD_MISO -> /GPIO23/MOSI
- U2 pad 19: Net-(U2-Pad19) -> unconnected-(U2-Pad19)
- U2 pad 21: Net-(U2-Pad19) -> unconnected-(U2-Pad19)
Other:
- board text removed: "by Hank"
