File: Demo/Egret.kicad_pcb (KiCad board)
At the start: 2 copper layers, 43.6 x 33.2 mm, 37 parts, among them Q1 S8050, Q2 S8050, Q3 AO3415AL, U1 WS2812B-B, U2 MPU6050, U3 LP2992IM5-3.3, U4 BH1750FVI-TR, U5 ESP32-PICO-D4, U6 AN2051-245_2.4G全向天线, U7 CP2102N-A01-GQFN28

Commit message: update
Parts:
- moved R7 7.11 mm to (121.6, 91.8), turned to 0 degrees
- moved U7 3.21 mm to (121.6, 87.5), turned to 0 degrees
- moved R6 1.79 mm to (121.9, 83.3), turned to 180 degrees
- moved U2 0.89 mm to (114.3, 86.8)
- moved Card1 0.09 mm to (125.1, 97.5)
- turned U3 to -90 degrees
Connections:
- net /USB-PWR-DM renamed /USB-PWR-DN
Routing:
- net +5V: track 0.00 -> 0.91 mm

Commit message: update
Parts:
- added ?: LOGO, G+D:logo, F.Cu at (136.9, 120.1)
- Card1, R10, R11, R12, R9: moved to F.Cu
- moved R10 28.1 mm to (124.6, 121.1), turned to 0 degrees
- moved R9 28.0 mm to (124.6, 118.1), turned to 0 degrees
- moved Card1 26.5 mm to (115.0, 122.0)
- moved R12 24.2 mm to (124.6, 123.0), turned to 0 degrees
- moved R11 23.8 mm to (124.6, 119.6), turned to 0 degrees
- moved U6 14.0 mm to (145.0, 112.5)
- moved R8 1.23 mm to (117.1, 97.8)
- moved C10 0.82 mm to (122.7, 97.8)
- moved C11 0.76 mm to (120.5, 97.8)
- moved C9 0.71 mm to (129.6, 107.0), turned to 0 degrees
- moved R1 0.71 mm to (129.6, 102.0)
- moved U4 0.71 mm to (129.6, 104.6)
- turned C5 to 180 degrees
- turned C3 to 180 degrees
- turned C4 to 180 degrees
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Routing:
- net +3V3: track 0.00 -> 162.1 mm, vias 0 -> 7
- net +5V: track 0.91 -> 70.4 mm, vias 0 -> 4
- net /GPIO4/RES: track 0.00 -> 48.6 mm, vias 0 -> 2
- net /GPIO26/SD_MISO: track 0.00 -> 47.5 mm, vias 0 -> 4
- net /GPIO14/SD_CLK: track 0.00 -> 43.5 mm, vias 0 -> 4
- net /GPIO33/MPU_SCL/BH_SCL: track 0.00 -> 41.9 mm, vias 0 -> 4
- net /GPIO32/MPU_SDA/BH_SDA: track 0.00 -> 41.3 mm, vias 0 -> 2
- net /GPIO13/SD_MOSI: track 0.00 -> 40.5 mm, vias 0 -> 4
- net /GPIO15/SD_CS: track 0.00 -> 39.5 mm, vias 0 -> 4
- net /GPIO18/SCK: track 0.00 -> 38.5 mm, vias 0 -> 3
- net /CP_Tx: track 0.00 -> 38.5 mm, vias 0 -> 2
- net /CP_Rx: track 0.00 -> 37.5 mm, vias 0 -> 2
- net /EN: track 0.00 -> 34.5 mm, vias 0 -> 3
- net /GPIO23/MOSI: track 0.00 -> 34.3 mm, vias 0 -> 4
- net /GPIO27/RGB_LED: track 0.00 -> 32.7 mm, vias 0 -> 2
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- added copper zone on B.Cu, net GND
- added copper zone on F.Cu, net GND
Other:
- board size 43.6 x 33.2 mm -> 43.6 x 50.3 mm

Commit message: update
Parts:
- moved ? 26.3 mm to (135.0, 123.0), turned to 180 degrees
- moved U6 4.73 mm to (145.0, 117.2)
- moved ? 3.42 mm to (135.0, 123.0), turned to 0 degrees
Routing:
- net /3V3A: track 21.6 -> 60.6 mm, vias 2 -> 8
- net Net-(U5-Pad2): track 2.35 -> 22.9 mm
- net /GPIO4/RES: track 48.6 -> 43.0 mm
- net /GPIO23/MOSI: track 34.3 -> 35.5 mm
- net +5V: track 70.4 -> 69.3 mm
- net /GPIO18/SCK: track 38.5 -> 39.5 mm, vias 3 -> 2
- net /EN: track 34.5 -> 35.5 mm
- net GND: vias 13 -> 2
- added copper zone on B.Cu, net (none)
- added copper zone on F.Cu, net (none)
- removed copper zone on B.Cu, net GND
- removed copper zone on F.Cu, net GND

Commit message: update
Parts:
- moved Card1 2.43 mm to (117.4, 121.8)
- moved R10 2.19 mm to (126.7, 122.0)
- moved R11 2.18 mm to (126.7, 120.4)
- moved R9 2.15 mm to (126.7, 118.8)
- moved R12 2.12 mm to (126.7, 123.6)
- moved ? 1.47 mm to (136.5, 123.0) (x2)
Routing:
- net +3V3: track 161.6 -> 168.8 mm
- net /GPIO26/SD_MISO: track 47.5 -> 51.4 mm
- net Net-(FPC1-Pad3): track 17.9 -> 20.5 mm
- net /GPIO14/SD_CLK: track 43.4 -> 45.5 mm
- net /GPIO15/SD_CS: track 39.5 -> 41.5 mm
- net /GPIO13/SD_MOSI: track 40.5 -> 41.7 mm
- net GND: vias 2 -> 3
Other:
- outline, holes or cut-outs redrawn

Commit message: update
Parts:
- moved R11 0.74 mm to (125.9, 120.4)
- moved R10 0.74 mm to (125.9, 122.0)
- moved R12 0.73 mm to (125.9, 123.6)
- moved R9 0.72 mm to (125.9, 118.8)
- moved ? 0.54 mm to (136.0, 123.1)
- moved ? 0.54 mm to (135.9, 123.1)
Routing:
- net /GPIO14/SD_CLK: track 45.5 -> 44.7 mm
- net /GPIO15/SD_CS: track 41.5 -> 40.8 mm
- net /GPIO26/SD_MISO: track 51.4 -> 50.7 mm
- net /GPIO13/SD_MOSI: track 41.7 -> 41.1 mm

Commit message: update
Parts:
- moved R9 3.23 mm to (126.1, 115.6)
- moved R11 2.03 mm to (126.1, 118.4)
- moved R12 0.76 mm to (126.1, 124.3)
- moved R10 0.63 mm to (126.1, 121.4)
- moved ? 0.10 mm to (136.1, 123.1)
- moved ? 0.10 mm to (136.0, 123.1)
- turned R5 to 180 degrees
Routing:
- net /GPIO5/LCD_BL: track 0.00 -> 27.1 mm, vias 0 -> 6
- net GND: track 0.00 -> 23.0 mm, vias 3 -> 4
- net +3V3: track 168.5 -> 176.7 mm
- net /RTS: track 7.21 -> 15.0 mm, vias 2 -> 3
- net Net-(Q3-Pad1): track 0.00 -> 3.45 mm
- net Net-(FPC1-Pad3): track 20.5 -> 17.5 mm, vias 1 -> 2
- net /USB-PWR-DN: track 17.7 -> 20.3 mm
- net /USB-PWR-DP: track 19.2 -> 21.2 mm
- net /3V3A: track 60.6 -> 58.9 mm
- net /GPIO18/SCK: track 39.5 -> 38.7 mm
- net +5V: track 69.3 -> 68.4 mm
- net /GPIO4/RES: track 43.0 -> 42.3 mm
- net /GPIO14/SD_CLK: track 44.7 -> 45.4 mm
- net /GPIO12: track 0.68 -> 0.00 mm, vias 1 -> 0
- net /GPIO15/SD_CS: track 40.8 -> 41.4 mm
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- added copper zone on B.Cu, net GND
- added copper zone on F.Cu, net GND
- removed copper zone on B.Cu, net (none)
- removed copper zone on F.Cu, net (none)
Other:
- board size 43.6 x 50.3 mm -> 43.7 x 50.3 mm

Commit message: update
Parts:
- moved C5 5.04 mm to (114.3, 83.4)
- moved C7 2.44 mm to (108.9, 83.4)
- moved C3 1.91 mm to (108.8, 86.1)
- moved C4 1.52 mm to (108.8, 88.7)
Routing:
- net GND: track 23.0 -> 84.4 mm, vias 4 -> 33
- net +3V3: track 176.7 -> 173.1 mm, vias 7 -> 6
- net Net-(C5-Pad1): track 9.92 -> 6.65 mm
- net +5V: track 68.4 -> 70.1 mm
- net Net-(C4-Pad1): track 4.51 -> 3.45 mm
- net Net-(U5-Pad2): track 22.9 -> 22.0 mm

Commit message: update
Routing:
- net GND: vias 33 -> 10
Changed lines of the file:
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@@
   (via (at 119.13 96.4) (size 0.8) (drill 0.4) (layers "F.Cu" "B.Cu") (net 9))
   (via (at 120.7 104.64) (size 0.9) (drill 0.7) (layers "F.Cu" "B.Cu") (net 9))
-  (via (at 129.75 109.51) (size 0.4) (drill 0.2) (layers "F.Cu" "B.Cu") (free) (net 9))
-  (via (at 133.04 112.89) (size 0.4) (drill 0.2) (layers "F.Cu" "B.Cu") (free) (net 9))
-  (via (at 132.26 112.07) (size 0.4) (drill 0.2) (layers "F.Cu" "B.Cu") (free) (net 9))
   (via (at 109.61 97.92) (size 0.8) (drill 0.4) (layers "F.Cu" "B.Cu") (net 9))
-  (via (at 130.18 109.94) (size 0.4) (drill 0.2) (layers "F.Cu" "B.Cu") (free) (net 9))
-  (via (at 124.66 106.36) (size 0.4) (drill 0.2) (layers "F.Cu" "B.Cu") (free) (net 9))
-  (via (at 128.8 108.55) (size 0.4) (drill 0.2) (layers "F.Cu" "B.Cu") (free) (net 9))
-  (via (at 125.31 107.52) (size 0.4) (drill 0.2) (layers "F.Cu" "B.Cu") (free) (net 9))
-  (via (at 131.02 110.82) (size 0.4) (drill 0.2) (layers "F.Cu" "B.Cu") (free) (net 9))
-  (via (at 131.46 111.26) (size 0.4) (drill 0.2) (layers "F.Cu" "B.Cu") (free) (net 9))
   (via (at 110.35 86.98) (size 0.4) (drill 0.2) (layers "F.Cu" "B.Cu") (net 9))
-  (via (at 133.42 113.27) (size 0.4) (drill 0.2) (layers "F.Cu" "B.Cu") (free) (net 9))
   (via (at 106.68 110.744) (size 0.8) (drill 0.4) (layers "F.Cu" "B.Cu") (net 9))
-  (via (at 124.48 107.34) (size 0.4) (drill 0.2) (layers "F.Cu" "B.Cu") (free) (net 9))
-  (via (at 128.3 108.1) (size 0.4) (drill 0.2) (layers "F.Cu" "B.Cu") (free) (net 9))
-  (via (at 127.82 107.63) (size 0.4) (drill 0.2) (layers "F.Cu" "B.Cu") (free) (net 9))
-  (via (at 130.63 110.4) (size 0.4) (drill 0.2) (layers "F.Cu" "B.Cu") (free) (net 9))
   (via (at 113.73 96.01) (size 0.8) (drill 0.4) (layers "F.Cu" "B.Cu") (net 9))
-  (via (at 131.87 111.67) (size 0.4) (drill 0.2) (layers "F.Cu" "B.Cu") (free) (net 9))
-  (via (at 126.7 106.83) (size 0.4) (drill 0.2) (layers "F.Cu" "B.Cu") (free) (net 9))
   (via (at 120.7 108.78) (size 0.7) (drill 0.5) (layers "F.Cu" "B.Cu") (net 9))
-  (via (at 133.82 113.63) (size 0.4) (drill 0.2) (layers "F.Cu" "B.Cu") (free) (net 9))
-  (via (at 129.28 109.04) (size 0.4) (drill 0.2) (layers "F.Cu" "B.Cu") (free) (net 9))
   (via (at 107.696 113.538) (size 0.8) (drill 0.4) (layers "F.Cu" "B.Cu") (net 9))
-  (via (at 125.33 106.39) (size 0.4) (drill 0.2) (layers "F.Cu" "B.Cu") (free) (net 9))
-  (via (at 134.22 114.01) (size 0.4) (drill 0.2) (layers "F.Cu" "B.Cu") (free) (net 9))
   (via (at 111.633542 88.673718) (size 0.4) (drill 0.2) (layers "F.Cu" "B.Cu") (net 9))
-  (via (at 126.04 106.55) (size 0.4) (drill 0.2) (layers "F.Cu" "B.Cu") (free) (net 9))
-  (via (at 132.66 112.52) (size 0.4) (drill 0.2) (layers "F.Cu" "B.Cu") (free) (net 9))
-  (via (at 127.28 107.2) (size 0.4) (drill 0.2) (layers "F.Cu" "B.Cu") (free) (net 9))
   (segment (start 110.35 86.98) (end 110.35 87.390176) (width 0.3) (layer "B.Cu") (net 9))
   (segment (start 120.7 108.78) (end 120.7 104.64) (width 0.4) (layer "B.Cu") (net 9))
