File: Hardware/Egret.kicad_pcb (KiCad board)
At the start: 2 copper layers, 10 parts, among them Q1 S8050, Q2 S8050, U1 AMS1117-3.3, U2 ESP32-PICO-D4, U3 CP2102N-A01-GQFN28

Commit message: generate PCB board
Parts:
- added C1: 10uF/25V (10%), Capacitor_SMD:C_0603_1608Metric, F.Cu at (123.5, 58.0)
- added C10: 0.1uF/25V (10%), Capacitor_SMD:C_0402_1005Metric, F.Cu at (123.8, 48.0)
- added C2: 0.1uF/25V (10%), Capacitor_SMD:C_0402_1005Metric, F.Cu at (123.8, 43.1)
- added C3: 0.1uF/25V (NC), Capacitor_SMD:C_0402_1005Metric, F.Cu at (164.5, 57.7)
- added C4: 10uF/25V (10%), Capacitor_SMD:C_0603_1608Metric, F.Cu at (155.4, 66.5)
- added C5: 4.7pF, Capacitor_SMD:C_0402_1005Metric, F.Cu at (173.4, 57.7)
- added C6: 2.7pF, Capacitor_SMD:C_0402_1005Metric, F.Cu at (127.2, 38.3)
- added C7: 0.1uF/25V, Capacitor_SMD:C_0402_1005Metric, F.Cu at (135.3, 41.3)
- added C8: 0.1uF/25V (10%), Capacitor_SMD:C_0402_1005Metric, F.Cu at (137.9, 46.2)
- added C9: 10uF/6.3V (10%), Capacitor_SMD:C_0402_1005Metric, F.Cu at (153.7, 46.2)
- added D1: Red LED, LED_SMD:LED_0603_1608Metric, F.Cu at (172.9, 52.6)
- added J1: Conn_01x20_Male, Connector_PinHeader_1.00mm:PinHeader_1x20_P1.00mm_Vertical, F.Cu at (138.0, 73.5)
- added J2: Conn_01x20_Male, Connector_PinHeader_1.00mm:PinHeader_1x20_P1.00mm_Vertical, F.Cu at (123.9, 73.5)
- added J3: USB_B_Micro, Connector_USB:USB_Micro-B_Molex-105017-0001, F.Cu at (121.7, 65.1)
- added L1: 1.6nH, Inductor_SMD:L_0402_1005Metric, F.Cu at (157.9, 36.4)
- added R1: 2k (1%), Resistor_SMD:R_0402_1005Metric, F.Cu at (175.3, 88.0)
- added R10: 0R (1%)(NC), Resistor_SMD:R_0402_1005Metric, F.Cu at (165.9, 46.1)
- added R11: 0R (1%)(NC), Resistor_SMD:R_0402_1005Metric, F.Cu at (164.2, 73.4)
- added R12: 10K (1%), Resistor_SMD:R_0402_1005Metric, F.Cu at (120.8, 38.3)
- added R13: 10K (1%), Resistor_SMD:R_0402_1005Metric, F.Cu at (170.3, 80.7)
- added R14: 0R (1%), Resistor_SMD:R_0402_1005Metric, F.Cu at (164.2, 37.6)
- added R15: 10K (1%)(NC), Resistor_SMD:R_0402_1005Metric, F.Cu at (163.7, 52.8)
- added R16: 22.1K(1%), Resistor_SMD:R_0402_1005Metric, F.Cu at (152.7, 41.3)
- added R17: 47.5K(1%), Resistor_SMD:R_0402_1005Metric, F.Cu at (144.0, 41.3)
- added R18: 0R (1%), Resistor_SMD:R_0402_1005Metric, F.Cu at (172.8, 73.4)
- added R2: 0.1uF/25V (10%), Resistor_SMD:R_0402_1005Metric, F.Cu at (123.8, 52.9)
- added R3: 10K (5%)(NC), Resistor_SMD:R_0402_1005Metric, F.Cu at (164.6, 92.9)
- added R4: 0R (1%), Resistor_SMD:R_0402_1005Metric, F.Cu at (143.2, 36.4)
- added R5: 0R (1%), Resistor_SMD:R_0402_1005Metric, F.Cu at (151.8, 36.4)
- added R6: 0R (1%), Resistor_SMD:R_0402_1005Metric, F.Cu at (134.4, 36.4)
- added R7: 2K (1%), Resistor_SMD:R_0402_1005Metric, F.Cu at (174.6, 46.1)
- added R8: 1K (1%), Resistor_SMD:R_0402_1005Metric, F.Cu at (173.8, 92.9)
- added R9: 1K (1%), Resistor_SMD:R_0402_1005Metric, F.Cu at (171.2, 37.6)
- added SW1: SW_Push, Button_Switch_SMD:SW_Push_SPST_NO_Alps_SKRK, F.Cu at (162.6, 79.4)
- added SW2: SW_Push, Button_Switch_SMD:SW_Push_SPST_NO_Alps_SKRK, F.Cu at (162.6, 86.7)
- Q1, Q2: footprint Package_TO_SOT_THT:TO-92_Inline -> Package_TO_SOT_SMD:SOT-23
- moved U2 104.8 mm to (154.8, 90.6), turned to 90 degrees
- moved U3 99.6 mm to (134.9, 65.5)
- moved E1 99.3 mm to (134.2, 52.5)
- moved Q2 92.7 mm to (169.1, 86.8)
- moved U1 91.9 mm to (152.4, 54.4)
- moved D3 84.7 mm to (155.6, 62.1)
- moved Q1 84.4 mm to (171.4, 67.0)
- moved D2 81.8 mm to (162.2, 62.1)
- moved D5 79.0 mm to (162.4, 42.1)
- moved D4 71.3 mm to (173.5, 42.0)
Connections:
- U3 pad 6: Net-(U3-Pad6) -> /VDD33
- U3 pad 7: Net-(U3-Pad6) -> /VDD33
Routing:
- net GND: track 0.00 -> 1.00 mm
Other:
- board outline added: 162 x 106 mm

Commit message: reorganize component locations
Parts:
- moved C10 444.3 mm to (567.3, 74.7)
- moved D4 433.2 mm to (522.0, 299.5)
- moved D5 430.9 mm to (533.4, 261.4)
- moved D3 430.4 mm to (522.0, 288.0)
- moved R10 426.5 mm to (475.9, 339.1)
- moved R14 424.3 mm to (531.5, 249.9)
- moved R9 420.4 mm to (475.9, 327.3)
- moved D2 418.9 mm to (522.0, 276.6)
- moved R18 418.5 mm to (550.5, 253.7)
- moved R11 414.5 mm to (475.9, 346.7)
- moved J3 411.8 mm to (487.7, 253.7)
- moved R17 404.8 mm to (547.1, 78.5)
- moved R16 394.5 mm to (547.1, 47.6)
- moved R12 381.5 mm to (476.2, 176.8)
- moved R8 377.7 mm to (475.9, 319.6)
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
Commit message: PCB layout
Parts:
- J1, J2: footprint Connector_PinHeader_1.00mm:PinHeader_1x20_P1.00mm_Vertical -> Connector_PinHeader_2.54mm:PinHeader_1x20_P2.54mm_Vertical
- moved R18 457.3 mm to (133.6, 65.8), turned to 180 degrees
- moved D4 449.2 mm to (133.8, 73.5)
- moved D3 444.5 mm to (133.7, 71.6)
- moved D5 444.2 mm to (133.7, 67.7)
- moved D2 439.9 mm to (133.7, 69.7)
- moved R14 439.1 mm to (133.6, 64.1), turned to 180 degrees
- moved R11 434.9 mm to (139.9, 70.6), turned to 180 degrees
- moved R10 429.0 mm to (139.9, 72.3), turned to 180 degrees
- moved C10 428.0 mm to (139.3, 78.2), turned to 180 degrees
- moved R9 424.9 mm to (139.9, 67.1), turned to 180 degrees
- moved R8 419.3 mm to (139.9, 68.8), turned to 180 degrees
- moved R17 419.0 mm to (128.1, 79.8), turned to 180 degrees
- moved R16 409.2 mm to (139.3, 81.0), turned to 180 degrees
- moved R15 407.8 mm to (128.1, 77.4), turned to 180 degrees
- moved J3 406.4 mm to (126.3, 67.8), turned to -90 degrees
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Routing:
- net GND: track 1.00 -> 0.00 mm
Other:
- board size 162 x 106 mm -> 92 x 37.2 mm

Commit message: update PCB
Parts:
- moved J1 51.2 mm to (152.7, 52.5), turned to 90 degrees
- moved C4 48.6 mm to (175.4, 61.1), turned to 180 degrees
- moved R7 41.2 mm to (167.7, 70.9), turned to 0 degrees
- moved R17 37.7 mm to (164.8, 71.0), turned to 0 degrees
- moved U1 36.4 mm to (169.0, 60.1), turned to 0 degrees
- moved R12 35.3 mm to (184.8, 63.7), turned to -90 degrees
- moved Q1 35.3 mm to (181.4, 63.5), turned to 180 degrees
- moved R13 35.3 mm to (184.8, 69.1)
- moved Q2 35.1 mm to (181.3, 68.9), turned to 180 degrees
- moved C7 35.0 mm to (181.8, 75.0)
- moved R5 35.0 mm to (185.8, 77.5)
- moved SW2 35.0 mm to (181.8, 77.6)
- moved R15 34.4 mm to (161.9, 71.0)
- moved R10 33.2 mm to (173.1, 71.8)
- moved R11 33.2 mm to (173.1, 70.0)
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Other:
- board size 92 x 37.2 mm -> 58.8 x 34.2 mm

Commit message: update PCB
Parts:
- moved R3 0.59 mm to (197.1, 76.8)
- moved R6 0.59 mm to (197.1, 58.5)
- moved R2 0.58 mm to (193.5, 76.8)
- moved E1 0.54 mm to (201.6, 72.3)
- moved C8 0.52 mm to (193.5, 58.5)
- turned U2 to -45 degrees

Commit message: update
Parts:
- J2: moved to B.Cu
- moved J2 47.6 mm to (200.2, 82.5)
- moved D4 9.88 mm to (155.7, 65.1)
- moved D3 5.08 mm to (155.7, 67.8)
- moved R1 4.03 mm to (162.1, 61.0), turned to 180 degrees
- moved C1 3.07 mm to (162.1, 62.4), turned to 180 degrees
- moved D5 2.49 mm to (155.9, 69.6)
- moved R18 2.36 mm to (155.9, 66.6)
- moved D1 2.33 mm to (162.1, 59.5)
- moved R14 1.69 mm to (155.9, 63.9)
- moved D2 1.46 mm to (155.7, 71.1)
- moved C4 1.04 mm to (175.7, 60.1), turned to 0 degrees
- turned C3 to 180 degrees
- turned R4 to 90 degrees
- turned SW1 to 180 degrees

Commit message: update
Parts:
- removed D2, D3, D4: LESD5D5.0CT1G, LESD5D5:TVS_LESD5D5.0CT1G
- removed D5: BAT760, BAT760:SOD323(F)
- removed E1: PRO-OB-440, PRO-OB-440:ANT_PRO-OB-440
- removed J3: USB_B_Micro, Connector_USB:USB_Micro-B_Molex-105017-0001
- removed R17: 47.5K(1%), Resistor_SMD:R_0402_1005Metric
- removed R18: 0R (1%), Resistor_SMD:R_0402_1005Metric
- added FPC1: FPC-05F-12PH20, Uinika.Footprint:FPC-SMD_12P-P0.50_FPC-05F-12PH20, F.Cu at (130.0, 58.8)
- added U4: CP2102-GMR-YJLTY, Uinika.Footprint:QFN-28_L5.0-W5.0-P0.50-TL-EP3.2-1, F.Cu at (139.8, 59.9)
- added U5: FPC-1.0FX-12PWBH20, Uinika.Footprint:FPC-SMD_12P-P1.00_XUNPU_FPC-1.0FX-12PWBH20, F.Cu at (114.8, 58.8)
- added U6: SD-CARD, Uinika.Footprint:TF-SMD_SD-CARD, F.Cu at (113.4, 72.4)
- added USB1: TYPEC-304J-BCP16, Uinika.Footprint:USB-C-SMD_TYPEC-304J-BCP16, F.Cu at (126.7, 67.8)
- C10, C8: footprint Capacitor_SMD:C_0402_1005Metric -> Capacitor_SMD:C_0603_1608Metric
- C2: value 0.1uF/25V (10%) -> 0.1uF/25V (NC); footprint Capacitor_SMD:C_0402_1005Metric -> Capacitor_SMD:C_0603_1608Metric
- C3: value 0.1uF/25V (NC) -> 10uF/25V (10%); footprint Capacitor_SMD:C_0402_1005Metric -> Capacitor_SMD:C_0603_1608Metric
- C4: value 10uF/25V (10%) -> 0.1uF/25V (10%)
- C5: value 4.7pF -> 2.7pF; footprint Capacitor_SMD:C_0402_1005Metric -> Capacitor_SMD:C_0603_1608Metric
- C6: value 2.7pF -> 10uF/6.3V (10%); footprint Capacitor_SMD:C_0402_1005Metric -> Capacitor_SMD:C_0603_1608Metric
- C7: value 0.1uF/25V -> 4.7pF; footprint Capacitor_SMD:C_0402_1005Metric -> Capacitor_SMD:C_0603_1608Metric
- C9: value 10uF/6.3V (10%) -> 0.1uF/25V; footprint Capacitor_SMD:C_0402_1005Metric -> Capacitor_SMD:C_0603_1608Metric
- R1, R6: footprint Resistor_SMD:R_0402_1005Metric -> Resistor_SMD:R_0603_1608Metric
- R10: value 0R (1%)(NC) -> 10K (1%); footprint Resistor_SMD:R_0402_1005Metric -> Resistor_SMD:R_0603_1608Metric
- R11: value 0R (1%)(NC) -> 2K (1%); footprint Resistor_SMD:R_0402_1005Metric -> Resistor_SMD:R_0603_1608Metric
- R12: value 10K (1%) -> 10K (1%)(NC); footprint Resistor_SMD:R_0402_1005Metric -> Resistor_SMD:R_0603_1608Metric
- R13: value 10K (1%) -> 1K (1%); footprint Resistor_SMD:R_0402_1005Metric -> Resistor_SMD:R_0603_1608Metric
- R14: value 0R (1%) -> 1K (1%); footprint Resistor_SMD:R_0402_1005Metric -> Resistor_SMD:R_0603_1608Metric
- R15: value 10K (1%)(NC) -> 0R (1%)(NC); footprint Resistor_SMD:R_0402_1005Metric -> Resistor_SMD:R_0603_1608Metric
- R16: value 22.1K(1%) -> 0R (1%)(NC); footprint Resistor_SMD:R_0402_1005Metric -> Resistor_SMD:R_0603_1608Metric
- R2: value 0.1uF/25V (10%) -> 0R (1%); footprint Resistor_SMD:R_0402_1005Metric -> Resistor_SMD:R_0603_1608Metric
- R3: value 10K (5%)(NC) -> 0R (1%); footprint Resistor_SMD:R_0402_1005Metric -> Resistor_SMD:R_0603_1608Metric
- R4: value 0R (1%) -> 0.1uF/25V (10%); footprint Resistor_SMD:R_0402_1005Metric -> Resistor_SMD:R_0603_1608Metric
- R5: value 0R (1%) -> 10K (5%)(NC); footprint Resistor_SMD:R_0402_1005Metric -> Resistor_SMD:R_0603_1608Metric
- R7: value 2K (1%) -> 47.5K(1%); footprint Resistor_SMD:R_0402_1005Metric -> Resistor_SMD:R_0603_1608Metric
- R8: value 1K (1%) -> 22.1K(1%); footprint Resistor_SMD:R_0402_1005Metric -> Resistor_SMD:R_0603_1608Metric
- R9: value 1K (1%) -> 10K (1%); footprint Resistor_SMD:R_0402_1005Metric -> Resistor_SMD:R_0603_1608Metric
- SW1, SW2: value SW_Push -> TD-1106SN-4.3H-160; footprint Button_Switch_SMD:SW_Push_SPST_NO_Alps_SKRK -> Uinika.Footprint:SW-SMD_L6.0-W3.3-LS8.0
- U1: footprint Package_TO_SOT_SMD:SOT-223-3_TabPin2 -> Uinika.Footprint:SOT-23-3_L2.9-W1.6-P1.90-LS2.9-BL
- U2: value ESP32-PICO-D4 -> AN2051-245_2.4G; footprint ESP32-PICO-D4:PQFN50P700X700X104-49N -> Uinika.Footprint:ANT-SMD_L5.0-W2.0
- U3: value CP2102N-A01-GQFN28 -> ESP32--PICO--D4; footprint CP2102N-A01-GQFN28:QFN50P500X500X80-29N -> Uinika.Footprint:QFN-48_L7.0-W7.0-P0.50-BL-EP5.4
Connections:
- C2 pad 1: /EN -> GND
- C2 pad 2: GND -> Net-(C2-Pad2)
- C3 pad 1: GND -> /VDD33
- C3 pad 2: Net-(C3-Pad2) -> GND
- C4 pad 1: /VDD33 -> Net-(C4-Pad1)
- C5 pad 1: /LNA_IN -> Net-(C5-Pad1)
- C5 pad 2: Net-(C5-Pad2) -> GND
- C6 pad 1: Net-(C5-Pad2) -> /VDD33A
- C7 pad 1: GND -> Net-(C7-Pad1)
- C7 pad 2: Net-(C7-Pad2) -> Net-(C5-Pad1)
- C9 pad 1: /VDD33A -> GND
- C9 pad 2: GND -> Net-(C9-Pad2)
- L1 pad 1: /LNA_IN -> Net-(C7-Pad1)
- R10 pad 1: /IO13 -> Net-(Q2-Pad2)
- R11 pad 1: /IO15 -> Net-(R11-Pad1)
- R11 pad 2: /CTS -> /VDD33
- R12 pad 1: Net-(Q1-Pad2) -> Net-(R12-Pad1)
- R12 pad 2: /DTR -> GND
- R13 pad 1: Net-(Q2-Pad2) -> /TXD0
- R13 pad 2: /RTS -> /RXD
- R14 pad 1: Net-(D4-Pad2) -> /RXD0
- R14 pad 2: /USB_DN -> /TXD
- R15 pad 1: Net-(R15-Pad1) -> /IO13
- R15 pad 2: GND -> /RTS
- R16 pad 1: /EXT_5V -> /IO15
- R16 pad 2: Net-(R16-Pad2) -> /CTS
- R2 pad 2: /EN -> /VDD33
- R3 pad 1: /IO12 -> Net-(C2-Pad2)
- R3 pad 2: /VDD33 -> /IO0
- R4 pad 1: Net-(C3-Pad2) -> /VDD33A
- R4 pad 2: /IO0 -> Net-(C4-Pad1)
- R5 pad 1: Net-(C7-Pad2) -> Net-(R5-Pad1)
- R5 pad 2: /EN -> /VDD33
- R6 pad 1: /VDD33A -> Net-(C9-Pad2)
- R6 pad 2: /VDD33 -> /EN
- R7 pad 1: Net-(R7-Pad1) -> GND
- R7 pad 2: /VDD33 -> Net-(R7-Pad2)
- R8 pad 1: /TXD0 -> /EXT_5V
- R8 pad 2: /RXD -> Net-(R7-Pad2)
- R9 pad 1: /RXD0 -> Net-(Q1-Pad2)
- R9 pad 2: /TXD -> /DTR
- SW1 pad 2: Net-(C3-Pad2) -> Net-(C2-Pad2)
- SW2 pad 2: Net-(C7-Pad2) -> Net-(C9-Pad2)
- U2 pad 1: /VDD33A -> Net-(C5-Pad1)
- U2 pad 2: /LNA_IN -> unconnected-(U2-Pad2)
- U3 pad 1: unconnected-(U3-Pad1) -> /VDD33A
- U3 pad 10: unconnected-(U3-Pad10) -> /IO34
- U3 pad 11: Net-(R15-Pad1) -> /IO35
- U3 pad 12: unconnected-(U3-Pad12) -> /IO32
- U3 pad 13: unconnected-(U3-Pad13) -> /IO33
- U3 pad 14: unconnected-(U3-Pad14) -> /IO25
- U3 pad 15: unconnected-(U3-Pad15) -> /IO26
- U3 pad 16: unconnected-(U3-Pad16) -> /IO27
- U3 pad 17: unconnected-(U3-Pad17) -> /IO14
- U3 pad 18: unconnected-(U3-Pad18) -> Net-(R5-Pad1)
- U3 pad 19: unconnected-(U3-Pad19) -> /VDD33A
- U3 pad 2: unconnected-(U3-Pad2) -> Net-(C7-Pad1)
- U3 pad 20: unconnected-(U3-Pad20) -> /IO13
- U3 pad 21: unconnected-(U3-Pad21) -> /IO15
- U3 pad 22: unconnected-(U3-Pad22) -> /IO2
- U3 pad 23: /CTS -> /IO0
- U3 pad 24: /RTS -> /IO4
- U3 pad 25: /RXD -> /FLASH_CS
- U3 pad 26: /TXD -> unconnected-(U3-Pad26)
- U3 pad 27: unconnected-(U3-Pad27) -> /FLASH_SD0
- U3 pad 28: /DTR -> /IO9
- U3 pad 29: GND -> /IO10
- U3 pad 3: GND -> /VDD33A
- U3 pad 4: /USB_DP -> /VDD33A
- U3 pad 5: /USB_DN -> /SENSOR_VP
- U3 pad 6: /VDD33 -> /IO37
- U3 pad 7: /VDD33 -> /IO38
- U3 pad 8: Net-(R16-Pad2) -> /SENSOR_VN
- U3 pad 9: Net-(R7-Pad1) -> Net-(C4-Pad1)

Commit message: update
Parts:
- added C11: 0.1uF/25V (10%), Capacitor_SMD:C_0603_1608Metric, F.Cu at (324.0, 61.2)
- added C12: 10nF, Capacitor_SMD:C_0603_1608Metric, F.Cu at (312.7, 5.34)
- added C13: 0.1uF, Capacitor_SMD:C_0603_1608Metric, F.Cu at (325.3, 17.1)
- added C14: 2.2nF, Capacitor_SMD:C_0603_1608Metric, F.Cu at (338.4, 80.6)
- added C15: 0.1uF, Capacitor_SMD:C_0603_1608Metric, F.Cu at (338.9, 54.2)
- added Card1: TF-02A_C2889261, Uinika.Footprint:TF-SMD_TF-02, F.Cu at (270.3, 44.9)
- added Q3: S8050, Package_TO_SOT_SMD:SOT-23, F.Cu at (336.1, 22.7)
- added R17: 0R (1%)(NC), Resistor_SMD:R_0603_1608Metric, F.Cu at (333.1, 9.74)
- added R18: 0R (1%)(NC), Resistor_SMD:R_0603_1608Metric, F.Cu at (321.6, 10.7)
- added R19: 10k, Resistor_SMD:R_0603_1608Metric, F.Cu at (340.8, 23.7)
- added R20: 10k, Resistor_SMD:R_0603_1608Metric, F.Cu at (340.2, 35.6)
- added R21: 10k, Resistor_SMD:R_0603_1608Metric, F.Cu at (340.2, 41.0)
- added R22: 10k, Resistor_SMD:R_0603_1608Metric, F.Cu at (340.2, 9.74)
- added U10: MPU6050-YJLTY, Uinika.Footprint:QFN-24_L4.0-W4.0-P0.50-BL-EP2.7, F.Cu at (314.8, 40.5)
- added U7: CP2102-GMR-YJLTY, Uinika.Footprint:QFN-28_L5.0-W5.0-P0.50-TL-EP3.2-1, F.Cu at (265.3, 25.1)
- added U9: FPC-1.0FX-12PWBH20, Uinika.Footprint:FPC-SMD_12P-P1.00_XUNPU_FPC-1.0FX-12PWBH20, F.Cu at (294.0, 40.0)
- C10: value 0.1uF/25V (10%) -> 0.1uF/25V
- C9: value 0.1uF/25V -> 0.1uF
- Q1: value S8050 -> AO3415AL; footprint Package_TO_SOT_SMD:SOT-23 -> Uinika.Footprint:SOT-23-3_L2.9-W1.6-P1.90-LS2.9-BL
- R10: value 10K (1%) -> 22.1K(1%)
- R11: value 2K (1%) -> 10K (1%)
- R12: value 10K (1%)(NC) -> 10K (1%)
- R13: value 1K (1%) -> 2K (1%)
- R14: value 1K (1%) -> 10K (1%)(NC)
- R15, R16: value 0R (1%)(NC) -> 1K (1%)
- R6: value 0R (1%) -> 10k
- R7: value 47.5K(1%) -> 0R (1%)
- R8: value 22.1K(1%) -> 1k
- R9: value 10K (1%) -> 47.5K(1%)
- SW1, SW2: value TD-1106SN-4.3H-160 -> TD-1106SN-5.0H-160; footprint Uinika.Footprint:SW-SMD_L6.0-W3.3-LS8.0 -> Uinika.Footprint:SW-SMD_L6.0-W3.3-LS8.0-1
- U1: value AMS1117-3.3 -> WS2812B-B; footprint Uinika.Footprint:SOT-23-3_L2.9-W1.6-P1.90-LS2.9-BL -> Uinika.Footprint:LED_WS2812B-B
- U2: value AN2051-245_2.4G -> AMS1117-3.3; footprint Uinika.Footprint:ANT-SMD_L5.0-W2.0 -> Uinika.Footprint:SOT-23-3_L2.9-W1.6-P1.90-LS2.9-BL
- U3: value ESP32--PICO--D4 -> AN2051-245_2.4G; footprint Uinika.Footprint:QFN-48_L7.0-W7.0-P0.50-BL-EP5.4 -> Uinika.Footprint:ANT-SMD_L5.0-W2.0
- U4: value CP2102-GMR-YJLTY -> BH1750FVI-TR; footprint Uinika.Footprint:QFN-28_L5.0-W5.0-P0.50-TL-EP3.2-1 -> Uinika.Footprint:XDCR_BH1750FVI-TR
- U5: value FPC-1.0FX-12PWBH20 -> ESP32--PICO--D4; footprint Uinika.Footprint:FPC-SMD_12P-P1.00_XUNPU_FPC-1.0FX-12PWBH20 -> Uinika.Footprint:QFN-48_L7.0-W7.0-P0.50-BL-EP5.4
- U6: value SD-CARD -> FPC-1.0FX-12PWBH20; footprint Uinika.Footprint:TF-SMD_SD-CARD -> Uinika.Footprint:FPC-SMD_12P-P1.00_XUNPU_FPC-1.0FX-12PWBH20
- moved U5 196.6 mm to (309.4, 30.9)
- moved R16 182.7 mm to (336.8, 16.3)
- moved U6 182.0 mm to (294.0, 49.7)
- moved R15 179.4 mm to (336.5, 29.7)
- moved R8 178.9 mm to (340.2, 4.34)
- moved R4 170.8 mm to (330.6, 19.4)
- moved D1 165.2 mm to (326.8, 45.3)
- moved R14 163.6 mm to (310.7, 10.7)
- moved R9 163.2 mm to (335.3, 48.2)
- moved R11 163.2 mm to (336.2, 75.2)
- moved FPC1 163.1 mm to (290.6, 30.9)
- moved U3 156.8 mm to (308.3, 15.3)
- moved C3 155.2 mm to (329.2, 80.6)
- moved R5 155.0 mm to (335.7, 38.0)
- moved U4 154.8 mm to (287.5, 13.6)
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Connections:
- C10 pad 1: /VDD33 -> GND
- C10 pad 2: GND -> Net-(C10-Pad2)
- C9 pad 1: GND -> +3V3
- C9 pad 2: Net-(C9-Pad2) -> GND
- Q1 pad 1: /RTS -> Net-(Q1-Pad1)
- Q1 pad 2: Net-(Q1-Pad2) -> +3V3
- Q1 pad 3: /EN -> Net-(Q1-Pad3)
- Q2 pad 1: /DTR -> Net-(Q2-Pad1)
- Q2 pad 3: /IO0 -> /EN
- R10 pad 1: Net-(Q2-Pad2) -> /EXT_5V
- R10 pad 2: /RTS -> Net-(R10-Pad2)
- R11 pad 1: Net-(R11-Pad1) -> Net-(Q2-Pad2)
- R11 pad 2: /VDD33 -> unconnected-(R11-Pad2)
- R12 pad 1: Net-(R12-Pad1) -> Net-(Q3-Pad2)
- R12 pad 2: GND -> Net-(Q2-Pad1)
- R13 pad 1: /TXD0 -> Net-(R13-Pad1)
- R13 pad 2: /RXD -> /VDD33
- R14 pad 1: /RXD0 -> Net-(R14-Pad1)
- R14 pad 2: /TXD -> GND
- R15 pad 1: /IO13 -> /TXD0
- R15 pad 2: /RTS -> /RXD
- R16 pad 1: /IO15 -> /RXD0
- R16 pad 2: /CTS -> /TXD
- R6 pad 1: Net-(C9-Pad2) -> Net-(R6-Pad1)
- R6 pad 2: /EN -> +3V3
- R7 pad 1: GND -> Net-(C10-Pad2)
- R7 pad 2: Net-(R7-Pad2) -> /EN
- R8 pad 1: /EXT_5V -> Net-(Q1-Pad1)
- R8 pad 2: Net-(R7-Pad2) -> /GPIO5/LCD_BL
- R9 pad 1: Net-(Q1-Pad2) -> GND
- R9 pad 2: /DTR -> Net-(R10-Pad2)
- SW2 pad 2: Net-(C9-Pad2) -> Net-(C10-Pad2)
- U1 pad 1: GND -> +5V
- U1 pad 2: /VDD33 -> unconnected-(U1-Pad2)
- U1 pad 3: Net-(C1-Pad1) -> GND
- U2 pad 1: Net-(C5-Pad1) -> GND
- U2 pad 2: unconnected-(U2-Pad2) -> /VDD33
- U3 pad 1: /VDD33A -> Net-(C5-Pad1)
- U3 pad 2: Net-(C7-Pad1) -> unconnected-(U3-Pad2)
- U4 pad 1: unconnected-(U4-Pad1) -> +3V3
- U4 pad 2: unconnected-(U4-Pad2) -> GND
- U4 pad 4: /USB_DP -> /GPIO32/MPU_SDA/BH_SDA
- U4 pad 5: /USB_DN -> Net-(R6-Pad1)
- U4 pad 6: /VDD33 -> /GPIO33/MPU_SCL/BH_SCL
- U5 pad 1: Net-(FPC1-Pad1) -> /VDD33A
- U5 pad 10: Net-(FPC1-Pad10) -> /IO34
- U5 pad 11: Net-(FPC1-Pad11) -> /IO35
- U5 pad 12: Net-(FPC1-Pad12) -> /IO32
- U5 pad 13: unconnected-(U5-Pad13) -> /IO33
- U5 pad 14: unconnected-(U5-Pad14) -> /IO25
- U5 pad 2: Net-(FPC1-Pad2) -> Net-(C7-Pad1)
- U5 pad 3: Net-(FPC1-Pad3) -> /VDD33A
- U5 pad 4: Net-(FPC1-Pad4) -> /VDD33A
- U5 pad 5: Net-(FPC1-Pad5) -> /SENSOR_VP
- U5 pad 6: Net-(FPC1-Pad6) -> /IO37
- U5 pad 7: Net-(FPC1-Pad7) -> /IO38
- U5 pad 8: Net-(FPC1-Pad8) -> /SENSOR_VN
- U5 pad 9: Net-(FPC1-Pad9) -> Net-(C4-Pad1)
- U6 pad 1: unconnected-(U6-Pad1) -> GND
- U6 pad 10: unconnected-(U6-Pad10) -> /GPIO23/MOSI
- U6 pad 11: unconnected-(U6-Pad11) -> /GPIO4/RES
- U6 pad 12: unconnected-(U6-Pad12) -> GND
- U6 pad 2: unconnected-(U6-Pad2) -> GND
- U6 pad 3: unconnected-(U6-Pad3) -> Net-(Q1-Pad3)
- U6 pad 4: unconnected-(U6-Pad4) -> +3V3
- U6 pad 5: unconnected-(U6-Pad5) -> GND
- U6 pad 6: unconnected-(U6-Pad6) -> GND
- U6 pad 7: unconnected-(U6-Pad7) -> /GPIO2/DC
- U6 pad 8: unconnected-(U6-Pad8) -> GND
- U6 pad 9: unconnected-(U6-Pad9) -> /GPIO18/SCK
