File: Hardware/Egret.kicad_pcb (KiCad board)
At the start: 2 copper layers, 58.8 x 34.2 mm, 58 parts, among them J1 Conn_01x20_Male, J2 Conn_01x20_Male, Q1 AO3415AL, Q2 S8050, Q3 S8050, SW1 TD-1106SN-5.0H-160, SW2 TD-1106SN-5.0H-160, U1 WS2812B-B, U10 MPU6050-YJLTY, U2 AMS1117-3.3, U3 AN2051-245_2.4G, U4 BH1750FVI-TR, U5 ESP32--PICO--D4, U6 FPC-1.0FX-12PWBH20, U7 CP2102-GMR-YJLTY, U9 FPC-1.0FX-12PWBH20

Commit message: update
Parts:
- J2: moved to F.Cu
- moved R20 230.7 mm to (125.8, 120.9)
- moved R8 228.8 mm to (133.9, 103.3), turned to 0 degrees
- moved R15 227.6 mm to (125.8, 115.9), turned to 0 degrees
- moved R19 225.0 mm to (125.8, 90.1)
- moved R22 224.3 mm to (129.8, 87.6)
- moved R5 222.9 mm to (125.8, 113.4), turned to 0 degrees
- moved R16 221.8 mm to (133.9, 105.8)
- moved C15 220.2 mm to (125.8, 109.8)
- moved R21 217.1 mm to (133.9, 108.4)
- moved R17 216.8 mm to (129.8, 85.1)
- moved R14 216.5 mm to (125.8, 123.4)
- moved R4 215.1 mm to (137.9, 114.9), turned to 0 degrees
- moved L1 214.6 mm to (125.3, 107.2), turned to 0 degrees
- moved C6 213.7 mm to (129.8, 110.9), turned to 0 degrees
- moved C9 213.4 mm to (137.9, 109.8), turned to 0 degrees
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Connections:
- C12 pad 1: +3V3 -> /VDD33
- C15 pad 1: +3V3 -> /VDD33
- C9 pad 1: +3V3 -> /VDD33
- Q1 pad 2: +3V3 -> /VDD33
- R6 pad 2: +3V3 -> /VDD33
- R8 pad 2: /GPIO5/LCD_BL -> /IO5
- U1 pad 1: +5V -> /EXT_5V
- U1 pad 4: /GPIO27/RGB_LED -> /IO27
- U10 pad 13: +3V3 -> /VDD33
- U10 pad 23: /GPIO33/MPU_SCL/BH_SCL -> /IO33
- U10 pad 24: /GPIO32/MPU_SDA/BH_SDA -> /IO32
- U10 pad 8: +3V3 -> /VDD33
- U4 pad 1: +3V3 -> /VDD33
- U4 pad 4: /GPIO32/MPU_SDA/BH_SDA -> /IO32
- U4 pad 6: /GPIO33/MPU_SCL/BH_SCL -> /IO33
- U6 pad 10: /GPIO23/MOSI -> /IO23
- U6 pad 11: /GPIO4/RES -> /IO4
- U6 pad 4: +3V3 -> /VDD33
- U6 pad 7: /GPIO2/DC -> /IO2
- U6 pad 9: /GPIO18/SCK -> /IO18
Other:
- board outline removed

Commit message: update
Parts:
- added C16: 10uF, Capacitor_SMD:C_0603_1608Metric, F.Cu at (140.1, 115.0)
- added C17: 0.1uF, Capacitor_SMD:C_0603_1608Metric, F.Cu at (134.8, 121.5)
- added C18: 10nF, Capacitor_SMD:C_0603_1608Metric, F.Cu at (152.2, 104.0)
- added J3: Conn_01x20_Male, Connector_PinHeader_2.54mm:PinHeader_1x20_P2.54mm_Vertical, F.Cu at (126.5, 74.3)
- added J4: Conn_01x20_Male, Connector_PinHeader_2.54mm:PinHeader_1x20_P2.54mm_Vertical, F.Cu at (121.8, 74.3)
- added U8: MPU6050-YJLTY, Uinika.Footprint:QFN-24_L4.0-W4.0-P0.50-BL-EP2.7, F.Cu at (143.2, 102.8)
- added USB2: TYPEC-304J-BCP16, Uinika.Footprint:USB-C-SMD_TYPEC-304J-BCP16, F.Cu at (134.2, 92.4)
- C1: value 10uF/25V (10%) -> 0.1uF/25V (NC)
- C10: value 0.1uF/25V -> 10uF/25V (10%)
- C2: value 0.1uF/25V (NC) -> 0.1uF/25V (10%)
- C3: value 10uF/25V (10%) -> 2.7pF
- C4: value 0.1uF/25V (10%) -> 10uF/6.3V (10%)
- C5: value 2.7pF -> 4.7pF
- C6: value 10uF/6.3V (10%) -> 0.1uF/25V (10%)
- C7: value 4.7pF -> 10uF/25V (10%)
- C8: value 0.1uF/25V (10%) -> 0.1uF
- C9: value 0.1uF -> 0.1uF/25V
- J1: value Conn_01x20_Male -> Conn_01x02_Male; footprint Connector_PinHeader_2.54mm:PinHeader_1x20_P2.54mm_Vertical -> Connector_PinHeader_2.54mm:PinHeader_1x02_P2.54mm_Vertical
- J2: value Conn_01x20_Male -> Conn_01x04_Male; footprint Connector_PinHeader_2.54mm:PinHeader_1x20_P2.54mm_Vertical -> Connector_PinHeader_2.54mm:PinHeader_1x04_P2.54mm_Vertical
- R1: value 2k (1%) -> 0R (1%)
- R10: value 22.1K(1%) -> 1K (1%)
- R11, R12: value 10K (1%) -> 0R (1%)(NC)
- R13: value 2K (1%) -> 47.5K(1%)
- R14: value 10K (1%)(NC) -> 22.1K(1%)
- R15: value 1K (1%) -> 2K (1%)
- R16: value 1K (1%) -> 10K (1%)(NC)
- R17, R18: value 0R (1%)(NC) -> 10K (1%)
- R3: value 0R (1%) -> 0.1uF/25V (10%)
- R4: value 0.1uF/25V (10%) -> 10K (5%)(NC)
- R5: value 10K (5%)(NC) -> 10k
- R6: value 10k -> 2k (1%)
- R9: value 47.5K(1%) -> 1K (1%)
- U10: value MPU6050-YJLTY -> FPC-1.0FX-12PWBH20; footprint Uinika.Footprint:QFN-24_L4.0-W4.0-P0.50-BL-EP2.7 -> Uinika.Footprint:FPC-SMD_12P-P1.00_XUNPU_FPC-1.0FX-12PWBH20
- U2: value AMS1117-3.3 -> AN2051-245_2.4G; footprint Uinika.Footprint:SOT-23-3_L2.9-W1.6-P1.90-LS2.9-BL -> Uinika.Footprint:ANT-SMD_L5.0-W2.0
- U3: value AN2051-245_2.4G -> BH1750FVI-TR; footprint Uinika.Footprint:ANT-SMD_L5.0-W2.0 -> Uinika.Footprint:XDCR_BH1750FVI-TR
- U4: value BH1750FVI-TR -> ESP32--PICO--D4; footprint Uinika.Footprint:XDCR_BH1750FVI-TR -> Uinika.Footprint:QFN-48_L7.0-W7.0-P0.50-BL-EP5.4
- U5: value ESP32--PICO--D4 -> AMS1117-3.3; footprint Uinika.Footprint:QFN-48_L7.0-W7.0-P0.50-BL-EP5.4 -> Uinika.Footprint:SOT-23-3_L2.9-W1.6-P1.90-LS2.9-BL
- U9: value FPC-1.0FX-12PWBH20 -> LP2992IM5-3.3; footprint Uinika.Footprint:FPC-SMD_12P-P1.00_XUNPU_FPC-1.0FX-12PWBH20 -> Uinika.Footprint:SOT95P280X145-5N
- moved R15 51.2 mm to (167.1, 85.5)
- moved C7 50.8 mm to (182.5, 80.4)
- moved J2 46.0 mm to (167.4, 74.3)
- moved R3 45.3 mm to (162.4, 99.3)
- moved C1 43.3 mm to (138.8, 81.0)
- moved R14 41.1 mm to (142.8, 86.0)
- moved R16 39.8 mm to (170.3, 89.7)
- moved C3 37.7 mm to (134.8, 81.0)
- moved C10 35.9 mm to (158.4, 99.3)
- moved C13 34.5 mm to (156.2, 104.0)
- moved R17 34.3 mm to (135.0, 119.0)
- moved R4 31.5 mm to (134.8, 83.5)
- moved R12 31.2 mm to (142.8, 81.0)
- moved R19 30.9 mm to (144.1, 115.0)
- moved C11 30.5 mm to (143.1, 117.5)
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Connections:
- C1 pad 1: Net-(C1-Pad1) -> GND
- C1 pad 2: GND -> Net-(C1-Pad2)
- C10 pad 1: GND -> /VDD33
- C10 pad 2: Net-(C10-Pad2) -> GND
- C2 pad 1: GND -> Net-(C2-Pad1)
- C2 pad 2: Net-(C2-Pad2) -> GND
- C3 pad 1: /VDD33 -> Net-(C3-Pad1)
- C4 pad 1: Net-(C4-Pad1) -> /VDD33A
- C5 pad 2: GND -> Net-(C3-Pad1)
- C7 pad 1: Net-(C7-Pad1) -> /EXT_5V
- C7 pad 2: Net-(C5-Pad1) -> GND
- C8 pad 1: /VDD33A -> /VDD33
- C9 pad 1: /VDD33 -> GND
- C9 pad 2: GND -> Net-(C9-Pad2)
- J1 pad 1: /FLASH_SD1 -> GND
- J1 pad 2: /FLASH_SD3 -> /VDD33
- J2 pad 1: /FLASH_CS -> +3V3
- J2 pad 2: /FLASH_SD0 -> GND
- J2 pad 3: /FLASH_SD2 -> /USB_CON+
- J2 pad 4: /SENSOR_VP -> /USB_CON-
- L1 pad 1: Net-(C7-Pad1) -> Net-(C5-Pad1)
- R1 pad 1: Net-(C1-Pad1) -> /VDD33A
- R1 pad 2: Net-(D1-Pad2) -> /VDD33
- R10 pad 1: /EXT_5V -> /RXD0
- R10 pad 2: Net-(R10-Pad2) -> /TXD
- R11 pad 1: Net-(Q2-Pad2) -> /IO13
- R11 pad 2: unconnected-(R11-Pad2) -> /RTS
- R12 pad 1: Net-(Q3-Pad2) -> /IO15
- R12 pad 2: Net-(Q2-Pad1) -> /CTS
- R13 pad 1: Net-(R13-Pad1) -> GND
- R13 pad 2: /VDD33 -> Net-(R13-Pad2)
- R14 pad 1: Net-(R14-Pad1) -> /EXT_5V
- R14 pad 2: GND -> Net-(R13-Pad2)
- R15 pad 1: /TXD0 -> Net-(R15-Pad1)
- R15 pad 2: /RXD -> /VDD33
- R16 pad 1: /RXD0 -> Net-(R16-Pad1)
- R16 pad 2: /TXD -> GND
- R17 pad 1: /IO13 -> Net-(Q2-Pad2)
- R17 pad 2: /RTS -> unconnected-(R17-Pad2)
- R18 pad 1: /IO15 -> Net-(Q3-Pad2)
- R18 pad 2: /CTS -> Net-(Q2-Pad1)
- R2 pad 1: /VDD33A -> Net-(C1-Pad2)
- R2 pad 2: /VDD33 -> /IO0
- R3 pad 1: Net-(C2-Pad2) -> /VDD33A
- R3 pad 2: /IO0 -> Net-(C2-Pad1)
- R4 pad 1: /VDD33A -> Net-(R4-Pad1)
- R4 pad 2: Net-(C4-Pad1) -> /VDD33
- R6 pad 1: Net-(R6-Pad1) -> /EXT_5V
- R6 pad 2: /VDD33 -> Net-(D1-Pad2)
- R7 pad 1: Net-(C10-Pad2) -> Net-(C9-Pad2)
- R9 pad 1: GND -> /TXD0
- R9 pad 2: Net-(R10-Pad2) -> /RXD
- SW1 pad 2: Net-(C2-Pad2) -> Net-(C1-Pad2)
- SW2 pad 2: Net-(C10-Pad2) -> Net-(C9-Pad2)
- U10 pad 1: GND -> Net-(FPC1-Pad1)
- U10 pad 10: Net-(C13-Pad2) -> Net-(FPC1-Pad10)
- U10 pad 11: GND -> Net-(FPC1-Pad11)
- U10 pad 12: unconnected-(U10-Pad12) -> Net-(FPC1-Pad12)
- U10 pad 13: /VDD33 -> unconnected-(U10-Pad13)
- U10 pad 2: unconnected-(U10-Pad2) -> Net-(FPC1-Pad2)
- U10 pad 3: unconnected-(U10-Pad3) -> Net-(FPC1-Pad3)
- U10 pad 4: unconnected-(U10-Pad4) -> Net-(FPC1-Pad4)
- U10 pad 5: unconnected-(U10-Pad5) -> Net-(FPC1-Pad5)
- U10 pad 6: unconnected-(U10-Pad6) -> Net-(FPC1-Pad6)
- U10 pad 7: unconnected-(U10-Pad7) -> Net-(FPC1-Pad7)
- U10 pad 8: /VDD33 -> Net-(FPC1-Pad8)
- U10 pad 9: GND -> Net-(FPC1-Pad9)
- U2 pad 1: GND -> Net-(C3-Pad1)
- U2 pad 2: /VDD33 -> unconnected-(U2-Pad2)
- U3 pad 1: Net-(C5-Pad1) -> /VDD33
- U3 pad 2: unconnected-(U3-Pad2) -> GND
- U4 pad 1: /VDD33 -> /VDD33A
- U4 pad 2: GND -> Net-(C5-Pad1)
- U4 pad 3: GND -> /VDD33A
- U4 pad 4: /IO32 -> /VDD33A
- U4 pad 5: Net-(R6-Pad1) -> /SENSOR_VP
- U4 pad 6: /IO33 -> /IO37
- U5 pad 1: /VDD33A -> GND
- U5 pad 2: Net-(C7-Pad1) -> /VDD33
- U5 pad 3: /VDD33A -> /EXT_5V
- U7 pad 11: Net-(R14-Pad1) -> Net-(R16-Pad1)
- U7 pad 8: Net-(R10-Pad2) -> Net-(R13-Pad2)
- U7 pad 9: Net-(R13-Pad1) -> Net-(R15-Pad1)
- U9 pad 1: Net-(FPC1-Pad1) -> /USB_5V
- U9 pad 2: Net-(FPC1-Pad2) -> GND
- U9 pad 3: Net-(FPC1-Pad3) -> /USB_5V
- U9 pad 4: Net-(FPC1-Pad4) -> Net-(C18-Pad1)
- U9 pad 5: Net-(FPC1-Pad5) -> +3V3

Commit message: update
Parts:
- moved C1 4.87 mm to (138.9, 76.1)
- moved C10 4.87 mm to (158.5, 94.4)
- moved C14 4.87 mm to (139.1, 115.2)
- moved C17 4.87 mm to (134.9, 116.6)
- moved C2 4.87 mm to (154.5, 101.6)
- moved C3 4.87 mm to (134.9, 76.1)
- moved C6 4.87 mm to (138.9, 81.2)
- moved C7 4.87 mm to (182.6, 75.5)
- moved C8 4.87 mm to (134.9, 81.2)
- moved C9 4.87 mm to (146.5, 105.1)
- moved D1 4.87 mm to (135.2, 111.6)
- moved FPC1 4.87 mm to (175.7, 69.5)
- moved Q1 4.87 mm to (131.0, 112.5)
- moved Q2 4.87 mm to (131.3, 108.0)
- moved Q3 4.87 mm to (141.7, 106.7)
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
Commit message: update
Parts:
- R11: value 0R (1%)(NC) -> 1K (1%)
- R13: value 47.5K(1%) -> 0R (1%)(NC)
- R9: value 1K (1%) -> 47.5K(1%)
- U7: value CP2102-GMR-YJLTY -> CP2102N-A02-GQFN28; footprint Uinika.Footprint:QFN-28_L5.0-W5.0-P0.50-TL-EP3.2-1 -> Uinika.Footprint:QFN-28_L5.0-W5.0-P0.50-TL-EP3.3
- moved U10 961.0 mm to (1067.8, 312.8)
- moved J4 949.6 mm to (1063.2, 194.7)
- moved C18 936.9 mm to (1062.9, -121.1)
- moved U9 915.8 mm to (1028.6, -104.0)
- moved R22 911.4 mm to (1037.7, 12.6)
- moved R19 902.1 mm to (1037.7, -13.3)
- moved R21 901.9 mm to (1037.7, 3.82)
- moved R20 893.5 mm to (1037.7, -4.55)
- moved C17 888.7 mm to (994.3, -109.7)
- moved Card1 881.1 mm to (1037.3, 61.7)
- moved J3 877.1 mm to (994.7, 194.7)
- moved FPC1 863.7 mm to (1004.9, 310.9)
- moved C16 863.6 mm to (975.2, -109.7)
- moved C15 786.2 mm to (875.4, 331.1)
- moved J2 780.5 mm to (924.9, -118.8)
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Connections:
- Q3 pad 1: unconnected-(Q3-Pad1) -> /DTR
- R10 pad 1: /RXD0 -> /TXD0
- R10 pad 2: /TXD -> /RXD
- R11 pad 1: /IO13 -> /RXD0
- R11 pad 2: /RTS -> /TXD
- R12 pad 1: /IO15 -> /IO13
- R12 pad 2: /CTS -> /RTS
- R13 pad 1: GND -> /IO15
- R13 pad 2: Net-(R13-Pad2) -> /CTS
- R14 pad 2: Net-(R13-Pad2) -> Net-(R14-Pad2)
- R17 pad 2: unconnected-(R17-Pad2) -> /DTR
- R9 pad 1: /TXD0 -> GND
- R9 pad 2: /RXD -> Net-(R14-Pad2)
Other:
- board outline added: 97.5 x 48 mm

Commit message: update
Connections:
- C16 pad 2: +3V3 -> Net-(C16-Pad2)
- C17 pad 2: +3V3 -> Net-(C16-Pad2)
- Card1 pad 1: unconnected-(Card1-Pad1) -> GND
- Card1 pad 2: /GPIO15/SD_CS -> unconnected-(Card1-Pad2)
- Card1 pad 3: /GPIO13/SD_MOSI -> /GPIO26/SD_MISO
- Card1 pad 4: +3V3 -> GND
- Card1 pad 6: GND -> /VDD33
- Card1 pad 7: /GPIO26/SD_MISO -> /GPIO13/SD_MOSI
- Card1 pad 8: unconnected-(Card1-Pad8) -> /GPIO15/SD_CS
- Card1 pad 9: GND -> unconnected-(Card1-Pad9)
- J2 pad 1: +3V3 -> Net-(C16-Pad2)
- Q2 pad 1: Net-(Q2-Pad1) -> /RTS
- R18 pad 2: Net-(Q2-Pad1) -> /RTS
- R19 pad 2: +3V3 -> /VDD33
- R20 pad 2: +3V3 -> /VDD33
- R21 pad 2: +3V3 -> /VDD33
- R22 pad 2: +3V3 -> /VDD33
- U7 pad 8: Net-(R13-Pad2) -> Net-(R14-Pad2)
- U9 pad 5: +3V3 -> Net-(C16-Pad2)

Commit message: update
Parts:
- moved C18 1010.4 mm to (75.7, 94.5)
- moved J4 1005.8 mm to (66.6, 59.2), turned to 90 degrees
- moved U10 994.8 mm to (96.0, 100.1), turned to 180 degrees
- moved U9 973.9 mm to (75.7, 97.2), turned to 180 degrees
- moved R19 939.4 mm to (100.8, 55.0), turned to -90 degrees
- moved C17 936.9 mm to (79.9, 94.8), turned to 180 degrees
- moved Card1 936.6 mm to (100.8, 46.7), turned to 180 degrees
- moved R21 936.4 mm to (102.7, 55.0), turned to -90 degrees
- moved R20 935.0 mm to (104.6, 55.0), turned to -90 degrees
- moved J3 933.5 mm to (67.0, 89.9), turned to 90 degrees
- moved R22 932.1 mm to (106.6, 55.0), turned to -90 degrees
- moved FPC1 932.1 mm to (96.0, 104.5)
- moved C16 919.0 mm to (79.9, 97.5), turned to 180 degrees
- moved J2 884.3 mm to (67.3, 96.5)
- moved C15 864.3 mm to (60.2, 43.9), turned to -90 degrees
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Connections:
- Card1 pad 3: /GPIO26/SD_MISO -> /IO26
- Card1 pad 5: /GPIO14/SD_CLK -> /IO14
- Card1 pad 7: /GPIO13/SD_MOSI -> /IO13
- Card1 pad 8: /GPIO15/SD_CS -> /IO15
- R19 pad 1: /GPIO26/SD_MISO -> /IO26
- R20 pad 1: /GPIO13/SD_MOSI -> /IO13
- R21 pad 1: /GPIO14/SD_CLK -> /IO14
- R22 pad 1: /GPIO15/SD_CS -> /IO15
- U10 pad 1: Net-(FPC1-Pad1) -> Net-(FPC1-Pad12)
- U10 pad 10: Net-(FPC1-Pad10) -> Net-(FPC1-Pad3)
- U10 pad 11: Net-(FPC1-Pad11) -> Net-(FPC1-Pad2)
- U10 pad 12: Net-(FPC1-Pad12) -> Net-(FPC1-Pad1)
- U10 pad 2: Net-(FPC1-Pad2) -> Net-(FPC1-Pad11)
- U10 pad 3: Net-(FPC1-Pad3) -> Net-(FPC1-Pad10)
- U10 pad 4: Net-(FPC1-Pad4) -> Net-(FPC1-Pad9)
- U10 pad 5: Net-(FPC1-Pad5) -> Net-(FPC1-Pad8)
- U10 pad 6: Net-(FPC1-Pad6) -> Net-(FPC1-Pad7)
- U10 pad 7: Net-(FPC1-Pad7) -> Net-(FPC1-Pad6)
- U10 pad 8: Net-(FPC1-Pad8) -> Net-(FPC1-Pad5)
- U10 pad 9: Net-(FPC1-Pad9) -> Net-(FPC1-Pad4)
Routing:
- net /IO2: track 0.00 -> 2.05 mm
- net (no net): vias 0 -> 4
Other:
- board size 97.5 x 48 mm -> 63.4 x 73.8 mm

Commit message: update
Parts:
- moved R18 20.0 mm to (94.4, 71.5), turned to 0 degrees
- moved Q2 16.1 mm to (94.4, 74.7), turned to -90 degrees
- moved R17 15.2 mm to (90.2, 71.5), turned to 180 degrees
- moved C1 13.5 mm to (79.6, 80.5), turned to 0 degrees
- moved SW1 13.3 mm to (81.2, 83.6), turned to 0 degrees
- moved SW2 10.5 mm to (92.4, 83.6), turned to 0 degrees
- moved C9 10.3 mm to (90.7, 80.4), turned to 0 degrees
- moved R7 10.3 mm to (93.9, 80.4), turned to 0 degrees
- moved Q3 9.68 mm to (90.2, 74.7), turned to -90 degrees
- moved R2 4.79 mm to (82.7, 80.5), turned to 0 degrees
- moved R5 4.20 mm to (79.7, 51.4)
- moved C8 4.20 mm to (74.8, 51.4)
- moved U3 4.20 mm to (77.2, 51.3)
- moved C14 3.65 mm to (60.3, 51.3)
- moved C15 3.53 mm to (63.2, 45.8)
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Routing:
- net /IO4: track 0.00 -> 2.05 mm
- net /IO2: track 2.05 -> 0.00 mm

Commit message: update
Parts:
- moved C7 3.04 mm to (65.3, 68.3), turned to 90 degrees
- moved J1 1.07 mm to (71.1, 69.5)
- moved D1 0.51 mm to (67.1, 68.3)
- moved R6 0.51 mm to (67.1, 65.0)
Changed lines of the file:
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@@
   )
   (setup
+    (stackup
+      (layer "F.SilkS" (type "Top Silk Screen"))
+      (layer "F.Paste" (type "Top Solder Paste"))
+      (layer "F.Mask" (type "Top Solder Mask") (thickness 0.01))
+      (layer "F.Cu" (type "copper") (thickness 0.035))
+      (layer "dielectric 1" (type "core") (thickness 1.51) (material "FR4") (epsilon_r 4.5) (loss_tangent 0.02))
+      (layer "B.Cu" (type "copper") (thickness 0.035))
+      (layer "B.Mask" (type "Bottom Solder Mask") (thickness 0.01))
+      (layer "B.Paste" (type "Bottom Solder Paste"))
+      (layer "B.SilkS" (type "Bottom Silk Screen"))
+      (copper_finish "None")
+      (dielectric_constraints no)
+    )
     (pad_to_mask_clearance 0)
     (pcbplotparams
@@
   )
   (footprint "Resistor_SMD:R_0603_1608Metric" (layer "F.Cu")
-    (at 66.548 65.024 -90)
+    (at 67.056 65.024 -90)
     (descr "Resistor SMD 0603 (1608 Metric), square (rectangular) end terminal, IPC_7351 nominal, (Body size source: IPC-SM-782 page 72, https://www.pcb-3d.com/wordpress/wp-content/uploads/ipc-sm-782a_amendment_1_and_2.pdf), generated with kicad-footprint-generator")
     (tags "resistor")
@@
   )
   (footprint "LED_SMD:LED_0603_1608Metric" (layer "F.Cu")
-    (at 66.568 68.264 90)
+    (at 67.076 68.264 90)
     (descr "LED SMD 0603 (1608 Metric), square (rectangular) end terminal, IPC_7351 nominal, (Body size source: http://www.tortai-tech.com/upload/download/2011102023233369053.pdf), generated with kicad-footprint-generator")
     (tags "LED")
@@
   )
   (footprint "Connector_PinHeader_2.54mm:PinHeader_1x02_P2.54mm_Vertical" (layer "F.Cu")
-    (at 72.183 69.484 90)
+    (at 71.115 69.484 90)
     (descr "Through hole straight pin header, 1x02, 2.54mm pitch, single row")
     (tags "Through hole pin header THT 1x02 2.54mm single row")
@@
   )
   (footprint "Capacitor_SMD:C_0603_1608Metric" (layer "F.Cu")
-    (at 68.318 68.284 -90)
+    (at 65.278 68.284 90)
     (descr "Capacitor SMD 0603 (1608 Metric), square (rectangular) end terminal, IPC_7351 nominal, (Body size source: IPC-SM-782 page 76, https://www.pcb-3d.com/wordpress/wp-content/uploads/ipc-sm-782a_amendment_1_and_2.pdf), generated with kicad-footprint-generator")
     (tags "capacitor")
@@
     (fp_line (start 0.8 -0.4) (end 0.8 0.4) (layer "F.Fab") (width 0.1))
     (fp_line (start -0.8 0.4) (end -0.8 -0.4) (layer "F.Fab") (width 0.1))
-    (pad "1" smd roundrect (at -0.775 0 270) (size 0.9 0.95) (layers "F.Cu" "F.Paste" "F.Mask") (roundrect_rratio 0.25)
+    (pad "1" smd roundrect (at -0.775 0 90) (size 0.9 0.95) (layers "F.Cu" "F.Paste" "F.Mask") (roundrect_rratio 0.25)
       (net 7 "/EXT_5V") (pintype "passive"))
-    (pad "2" smd roundrect (at 0.775 0 270) (size 0.9 0.95) (layers "F.Cu" "F.Paste" "F.Mask") (roundrect_rratio 0.25)
+    (pad "2" smd roundrect (at 0.775 0 90) (size 0.9 0.95) (layers "F.Cu" "F.Paste" "F.Mask") (roundrect_rratio 0.25)
       (net 1 "GND") (pintype "passive"))
     (model "${KICAD6_3DMODEL_DIR}/Capacitor_SMD.3dshapes/C_0603_1608Metric.wrl"
