File: Hardware/Egret.kicad_pcb (KiCad board)
At the start: 2 copper layers, 64.6 x 69.3 mm, 56 parts, among them Q1 S8050, Q2 S8050, Q3 AO3415AL, SW1 TD-1106SN-5.0H-160, SW2 TD-1106SN-5.0H-160, U1 WS2812B-B, U10 ST7789_FPC_PAD, U2 AN2051-245_2.4G, U3 ESP32--PICO--D4, U4 MPU6050-YJLTY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

Commit message: update
Parts:
- added ?: LOGO, Uinika.Footprint:G+D-small, F.Cu at (179.1, 95.1)
- added ?: LOGO, Uinika.Footprint:G+D-big, F.Cu at (148.3, 125.1)
- added ?: LOGO, Uinika.Footprint:G+D-big, B.Cu at (148.2, 125.1)
- added ?: LOGO, Uinika.Footprint:G+D-big, B.Cu at (166.3, 87.2)
- Q3, R18, U10, U9: moved to B.Cu
- moved R18 9.86 mm to (150.3, 111.9), turned to 180 degrees
- moved U10 9.82 mm to (150.3, 109.4), turned to 0 degrees
- moved Q3 9.73 mm to (150.2, 118.8), turned to 0 degrees
- moved U9 7.59 mm to (145.7, 115.6)
- turned C7 to 0 degrees
Connections:
- U3 pad : (no net) -> GND
Routing:
- net GND: track 118.9 -> 184.2 mm, vias 9 -> 26
- net /VDD33: track 100.4 -> 135.9 mm, vias 3 -> 4
- net /IO0: track 22.0 -> 44.2 mm, vias 2 -> 6
- net /VDD33A: track 34.0 -> 53.9 mm, vias 3 -> 5
- net Net-(D1-Pad2): track 0.00 -> 10.0 mm, vias 0 -> 2
- net /EXT_5V: track 60.7 -> 63.0 mm
- net /IO18: track 21.9 -> 20.1 mm
- net /IO4: track 14.0 -> 15.1 mm
- net /IO2: track 17.3 -> 18.2 mm
- net /IO13: vias 5 -> 4
- net (no net): vias 8 -> 0
Other:
- board size 64.6 x 69.3 mm -> 64.6 x 60.3 mm
- board text added: "Giesecke+Devrient"
- board text added: "Version 0.0.2"

Commit message: update
Parts:
- moved C15 8.39 mm to (129.8, 87.0), turned to -90 degrees
Routing:
- net /VDD33: track 135.9 -> 133.5 mm
- net /IO2: track 18.2 -> 15.9 mm
- net GND: track 184.2 -> 182.3 mm, vias 26 -> 27

Commit message: update
Parts:
- moved ? 0.20 mm to (166.3, 87.0)
Changed lines of the file:
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@@
   )
   (footprint "Uinika.Footprint:G+D-big" (layer "F.Cu")
-    (at 148.273859 125.145001)
+    (at 148.293859 125.105001)
     (attr board_only exclude_from_pos_files exclude_from_bom)
     (fp_text reference "" (at 0 0) (layer "F.SilkS")
@@
   )
   (footprint "Uinika.Footprint:G+D-big" (layer "B.Cu")
-    (at 148.23 125.13 180)
+    (at 148.25 125.09 180)
     (attr board_only exclude_from_pos_files exclude_from_bom)
     (fp_text reference "" (at 0 0) (layer "B.SilkS")
@@
   )
   (footprint "Uinika.Footprint:G+D-big" (layer "B.Cu")
-    (at 166.304999 87.196141 -90)
+    (at 166.3 87 -90)
     (attr board_only exclude_from_pos_files exclude_from_bom)
     (fp_text reference "" (at 0 0 90) (layer "B.SilkS")
@@
     (effects (font (size 0.5 0.5) (thickness 0.1)) (justify mirror))
   )
-  (gr_text "Giesecke+Devrient" (at 171.29 86.63 90) (layer "B.SilkS")
+  (gr_text "Giesecke+Devrient" (at 171.6 86.63 90) (layer "B.SilkS")
     (effects (font (size 1.3 1.3) (thickness 0.2)) (justify mirror))
   )
@@
     (effects (font (size 0.5 0.5) (thickness 0.1)) (justify mirror))
   )
-  (gr_text "Giesecke+Devrient" (at 148.35 130.41) (layer "B.SilkS")
+  (gr_text "Giesecke+Devrient" (at 148.62 130.36) (layer "B.SilkS")
     (effects (font (size 1.3 1.3) (thickness 0.2)) (justify mirror))
   )
@@
     (effects (font (size 0.5 0.5) (thickness 0.1)))
   )
-  (gr_text "Giesecke+Devrient" (at 148.32 130.43) (layer "F.SilkS")
+  (gr_text "Giesecke+Devrient" (at 148.02 130.36) (layer "F.SilkS")
     (effects (font (size 1.3 1.3) (thickness 0.2)))
   )

Commit message: update
Parts:
- moved SW2 0.95 mm to (142.4, 97.1)
- moved C10 0.90 mm to (147.8, 97.1)
- moved R6 0.87 mm to (137.0, 97.1)
Routing:
- net /EN: track 15.9 -> 15.1 mm
- net GND: track 182.3 -> 181.6 mm

Commit message: update
Parts:
- moved R9 0.61 mm to (145.3, 80.9)
- moved R8 0.59 mm to (145.3, 82.5)
- moved R10 0.57 mm to (145.3, 84.0)
- moved R11 0.55 mm to (145.3, 85.6)
- moved R17 0.53 mm to (142.9, 92.6)
- moved R16 0.47 mm to (142.9, 89.1)
- moved Q2 0.31 mm to (146.2, 92.6)
- moved Q1 0.25 mm to (146.2, 89.0)
Routing:
- net /RTS: track 23.7 -> 29.4 mm
- net GND: track 181.6 -> 184.9 mm, vias 27 -> 26
- net /IO5: track 16.8 -> 18.3 mm
- net /RXD0: track 38.1 -> 39.3 mm
- net /IO23: track 23.2 -> 24.2 mm
- net /EN: track 15.1 -> 15.9 mm
- net /IO27: track 24.3 -> 25.1 mm
- net /VDD33: track 133.5 -> 134.2 mm
- net /TXD0: track 39.4 -> 40.1 mm
- net Net-(Q2-Pad2): track 1.76 -> 2.42 mm
- net Net-(Q1-Pad2): track 2.69 -> 3.34 mm

Commit message: update
Parts:
- moved U2 0.19 mm to (179.7, 86.9)
Routing:
- net Net-(C3-Pad1): track 5.02 -> 5.62 mm
Changed lines of the file:
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@@
   )
   (footprint "Uinika.Footprint:ANT-SMD_L5.0-W2.0" (layer "F.Cu")
-    (at 179.62 87.08 90)
+    (at 179.7 86.91 90)
     (property "Sheetfile" "Egret.kicad_sch")
     (property "Sheetname" "")
@@
   (segment (start 168.519233 83.003) (end 168.13099 83.391243) (width 0.4) (layer "F.Cu") (net 3))
   (segment (start 172.407 82.988) (end 172.905 82.49) (width 0.4) (layer "F.Cu") (net 3))
-  (segment (start 176.545 87.0875) (end 179.0375 89.58) (width 0.3) (layer "F.Cu") (net 4))
+  (segment (start 178.8675 89.41) (end 179.7 89.41) (width 0.3) (layer "F.Cu") (net 4))
+  (segment (start 176.545 87.0875) (end 178.8675 89.41) (width 0.3) (layer "F.Cu") (net 4))
   (segment (start 176.545 85.5875) (end 176.545 87.0875) (width 0.3) (layer "F.Cu") (net 4))
   (segment (start 169.19165 89.06165) (end 169.997 89.867) (width 0.4) (layer "F.Cu") (net 5))

Commit message: update
Parts:
- moved U1 0.19 mm to (155.2, 97.0)
