File: Hardware/Egret.kicad_sch (KiCad schematic)
At the start: 45 parts, among them J1 Conn_01x20_Male, J2 Conn_01x20_Male, J3 USB_B_Micro, Q1 S8050, Q2 S8050, SW1 SW_Push, SW2 SW_Push, U1 AMS1117-3.3, U2 ESP32-PICO-D4, U3 CP2102N-A01-GQFN28

Commit message: fix some bugs
Parts:
- C1: value 10uF/25V(10%) -> 10uF/25V (10%)
- C10: value 0.1uF/25V(10%) -> 0.1uF/25V (10%)
- C2: value C -> 0.1uF/25V (10%)
- C5: value C -> 4.7pF
- C6: renamed from C7; value C -> 2.7pF
- C8: renamed from C6; value 0.1uF/25V(10%) -> 0.1uF/25V (10%)
- D2, D3, D4: footprint TVS_LESD5D5.0CT1G -> LESD5D5:TVS_LESD5D5.0CT1G
- D5: footprint SOD323(F) -> BAT760:SOD323(F)
- E1: footprint ANT_PRO-OB-440 -> PRO-OB-440:ANT_PRO-OB-440
- L1: value L -> 1.6nH
- R10, R11: value 0R(1%)(NC) -> 0R (1%)(NC)
- R15: renamed from R17; value 10K(1%)(NC) -> 10K (1%)(NC)
- R18: value 0R(1%) -> 0R (1%)
- R2: renamed from R3; value 0.1uF/25V(10%) -> 0.1uF/25V (10%)
- R8, R9: value 1K(1%) -> 1K (1%)
- U2: footprint PQFN50P700X700X104-49N -> ESP32-PICO-D4:PQFN50P700X700X104-49N
- U3: footprint QFN50P500X500X80-29N -> CP2102N-A01-GQFN28:QFN50P500X500X80-29N
- renumbered C8 to C7, R15 to R16, R16 to R17, R2 to R3
Connections:
- net VDD33: now also C10.1, U3.6 (VDD), U3.7 (VREGIN)
Other:
- moved on the sheet: C2, C8, C9, R2, R6

Commit message: generate PCB board
Parts:
- C1, C4: footprint (none) -> Capacitor_SMD:C_0603_1608Metric
- C10, C2, C3, C5, C6, C7, C8, C9: footprint (none) -> Capacitor_SMD:C_0402_1005Metric
- D1: footprint (none) -> LED_SMD:LED_0603_1608Metric
- J1, J2: footprint (none) -> Connector_PinHeader_1.00mm:PinHeader_1x20_P1.00mm_Vertical
- J3: footprint (none) -> Connector_USB:USB_Micro-B_Molex-105017-0001
- L1: footprint (none) -> Inductor_SMD:L_0402_1005Metric
- Q1, Q2: footprint Package_TO_SOT_THT:TO-92_Inline -> Package_TO_SOT_SMD:SOT-23
- R1, R10, R11, R12, R13, R14, R15, R16, R17, R18, R2, R3, R4, R5, R6, R7, R8, R9: footprint (none) -> Resistor_SMD:R_0402_1005Metric
- SW1, SW2: footprint (none) -> Button_Switch_SMD:SW_Push_SPST_NO_Alps_SKRK

Commit message: PCB layout
Parts:
- J1, J2: footprint Connector_PinHeader_1.00mm:PinHeader_1x20_P1.00mm_Vertical -> Connector_PinHeader_2.54mm:PinHeader_1x20_P2.54mm_Vertical
Changed lines of the file:
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@@
       (effects (font (size 1.27 1.27)) (justify right))
     )
-    (property "Footprint" "Connector_PinHeader_1.00mm:PinHeader_1x20_P1.00mm_Vertical" (id 2) (at 223.52 50.8 0)
+    (property "Footprint" "Connector_PinHeader_2.54mm:PinHeader_1x20_P2.54mm_Vertical" (id 2) (at 223.52 50.8 0)
       (effects (font (size 1.27 1.27)) hide)
     )
@@
     (property "Reference" "J1" (id 0) (at 180.594 23.876 0))
     (property "Value" "Conn_01x20_Male" (id 1) (at 179.832 80.264 0))
-    (property "Footprint" "Connector_PinHeader_1.00mm:PinHeader_1x20_P1.00mm_Vertical" (id 2) (at 177.8 50.8 0)
+    (property "Footprint" "Connector_PinHeader_2.54mm:PinHeader_1x20_P2.54mm_Vertical" (id 2) (at 177.8 50.8 0)
       (effects (font (size 1.27 1.27)) hide)
     )
@@
     )
     (path "/9832501f-af9f-4986-a2cc-35159569a913"
-      (reference "J1") (unit 1) (value "Conn_01x20_Male") (footprint "Connector_PinHeader_1.00mm:PinHeader_1x20_P1.00mm_Vertical")
+      (reference "J1") (unit 1) (value "Conn_01x20_Male") (footprint "Connector_PinHeader_2.54mm:PinHeader_1x20_P2.54mm_Vertical")
     )
     (path "/5fac6571-5859-4377-9596-fb4b76d22263"
-      (reference "J2") (unit 1) (value "Conn_01x20_Male") (footprint "Connector_PinHeader_1.00mm:PinHeader_1x20_P1.00mm_Vertical")
+      (reference "J2") (unit 1) (value "Conn_01x20_Male") (footprint "Connector_PinHeader_2.54mm:PinHeader_1x20_P2.54mm_Vertical")
     )
     (path "/b9ddff79-f037-427e-acab-acd7cbf8fd2e"

Commit message: update
Parts:
- removed C2: 0.1uF/25V (10%), Capacitor_SMD:C_0402_1005Metric, symbol Device:C
- removed C9: 10uF/6.3V (10%), Capacitor_SMD:C_0402_1005Metric, symbol Device:C
- removed D2, D3, D4: LESD5D5.0CT1G, LESD5D5:TVS_LESD5D5.0CT1G, symbol LESD5D5.0CT1G:LESD5D5.0CT1G
- removed D5: BAT760, BAT760:SOD323(F), symbol BAT760:BAT760
- removed E1: PRO-OB-440, PRO-OB-440:ANT_PRO-OB-440, symbol PRO-OB-440:PRO-OB-440
- removed J3: USB_B_Micro, Connector_USB:USB_Micro-B_Molex-105017-0001, symbol Connector:USB_B_Micro
- removed R14, R18, R6: 0R (1%), Resistor_SMD:R_0402_1005Metric, symbol Device:R
- removed R15: 10K (1%)(NC), Resistor_SMD:R_0402_1005Metric, symbol Device:R
- removed R16: 22.1K(1%), Resistor_SMD:R_0402_1005Metric, symbol Device:R
- removed R17: 47.5K(1%), Resistor_SMD:R_0402_1005Metric, symbol Device:R
- removed R3: 10K (5%)(NC), Resistor_SMD:R_0402_1005Metric, symbol Device:R
- removed SW1, SW2: SW_Push, Button_Switch_SMD:SW_Push_SPST_NO_Alps_SKRK, symbol Switch:SW_Push
- removed U2: ESP32-PICO-D4, ESP32-PICO-D4:PQFN50P700X700X104-49N, symbol ESP32-PICO-D4:ESP32-PICO-D4
- removed U3: CP2102N-A01-GQFN28, CP2102N-A01-GQFN28:QFN50P500X500X80-29N, symbol CP2102N-A01-GQFN28:CP2102N-A01-GQFN28
- added C4: 0.1uF/25V (10%), Capacitor_SMD:C_0402_1005Metric, symbol Device:C
- added C7: 4.7pF, Capacitor_SMD:C_0402_1005Metric, symbol Device:C
- added FPC1: FPC-05F-12PH20, kicad_lceda:FPC-SMD_12P-P0.50_FPC-05F-12PH20, symbol Uinika:FPC-05F-12PH20
- added R11: 2K (1%), Resistor_SMD:R_0402_1005Metric, symbol Device:R
- added R12: 10K (1%)(NC), Resistor_SMD:R_0402_1005Metric, symbol Device:R
- added R4: 0.1uF/25V (10%), Resistor_SMD:R_0402_1005Metric, symbol Device:R
- added R5: 10K (5%)(NC), Resistor_SMD:R_0402_1005Metric, symbol Device:R
- added R8: 22.1K(1%), Resistor_SMD:R_0402_1005Metric, symbol Device:R
- added SW1, SW2: TD-1106SN-4.3H-160, kicad_lceda:SW-SMD_L6.0-W3.3-LS8.0, symbol Uinika:TD-1106SN-4.3H-160
- added U2: AN2051-245_2.4G, kicad_lceda:ANT-SMD_L5.0-W2.0, symbol Uinika:AN2051-245_2.4G
- added U3: ESP32--PICO--D4, kicad_lceda:QFN-48_L7.0-W7.0-P0.50-BL-EP5.4, symbol Uinika:ESP32--PICO--D4
- added U4: CP2102-GMR-YJLTY, kicad_lceda:QFN-28_L5.0-W5.0-P0.50-TL-EP3.2-1, symbol Uinika:CP2102-GMR-YJLTY
- added U5: FPC-1.0FX-12PWBH20, kicad_lceda:FPC-SMD_12P-P1.00_XUNPU_FPC-1.0FX-12PWBH20, symbol Uinika:FPC-1.0FX-12PWBH20
- added USB1: TYPEC-304J-BCP16, kicad_lceda:USB-C-SMD_TYPEC-304J-BCP16, symbol Uinika:TYPEC-304J-BCP16
- C5: value 4.7pF -> 2.7pF
- C6: value 2.7pF -> 10uF/6.3V (10%)
- R2: value 0.1uF/25V (10%) -> 0R (1%)
- R7: value 2K (1%) -> 47.5K(1%)
- renumbered C3 to C2, C4 to C3, C7 to C9, R13 to R10, R8 to R13, R9 to R14, R10 to R15, R11 to R16, R4 to R3, R5 to R6, R12 to R9
Connections:
- net CTS: now also U4.23 (CTS)
- net DTR: now also U4.28 (DTR)
- net EN: no longer R2.2
- net EXT_5V: now also R8.1, USB1.A4B9 (VBUS), USB1.B4A9 (VBUS)
- net FLASH_CLK: now also U3.31 (CLK)
- net FLASH_CS: now also U3.25 (IO16)
- net FLASH_SD0: now also U3.27 (IO17)
- net FLASH_SD1: now also U3.33 (SD1)
- net FLASH_SD2: now also U3.30 (CMD)
- net FLASH_SD3: now also U3.32 (SD0)
- net GND: now also C5.2, R7.1, C4.2, R12.2, SW1.1, SW2.1, U3.49 (GND), U4.29 (GND), U4.3 (GND), U4.30 (GND), USB1.13 (GND), USB1.14 (GND), USB1.15 (GND), USB1.16 (GND), USB1.A1B12 (GND), USB1.B1A12 (GND)
- net IO0: now also U3.23 (IO0)
- net IO10: now also U3.29 (SD3)
- net IO13: now also U3.20 (IO13)
- net IO14: now also U3.17 (IO14)
- net IO15: now also U3.21 (IO15)
- net IO18: now also U3.35 (IO18)
- net IO19: now also U3.38 (IO19)
- net IO2: now also U3.22 (IO2)
- net IO21: now also U3.42 (IO21)
- net IO22: now also U3.39 (IO22)
- net IO23: now also U3.36 (IO23)
- net IO25: now also U3.14 (IO25)
- net IO26: now also U3.15 (IO26)
- net IO27: now also U3.16 (IO27)
- net IO32: now also U3.12 (IO32)
- net IO33: now also U3.13 (IO33)
- net IO34: now also U3.10 (IO34)
- net IO35: now also U3.11 (IO35)
- net IO37: now also U3.6 (SENSOR_CAPP)
- net IO38: now also U3.7 (SENSOR_CAPN)
- net IO4: now also U3.24 (IO4)
- net IO5: now also U3.34 (IO5)
- net IO9: now also U3.28 (SD2)
- net RTS: now also U4.24 (RTS)
- net RXD: now also U4.25 (RXD)
- net RXD0: now also U3.40 (U0RXD)
- net SENSOR_VN: now also U3.8 (SENSOR_VN)
- net SENSOR_VP: now also U3.5 (SENSOR_VP)
- net TXD: now also U4.26 (TXD)
- net TXD0: now also U3.41 (U0TXD)
- net USB_DN: now also U4.5 (D-), USB1.A7 (DN1), USB1.B7 (DN2)
- net USB_DP: now also U4.4 (D+), USB1.A6 (DP1), USB1.B6 (DP2)
- net VDD33: now also R2.2, R11.2, R5.2, U4.6 (DD), U4.7 (REGIN); no longer R7.2
- net VDD33A: now also C6.1, R4.1, U3.1 (VDDA), U3.19 (VDD3P3_RTC), U3.3 (VDDA3P3), U3.37 (VDD3P3_CPU), U3.4 (VDDA3P3), U3.43 (VDDA), U3.46 (VDDA)
- net at C2.2, R3.1: now also SW1.2
- net at C9.2, R6.1: now also SW2.2
- net LNA_IN: no longer names the net of L1.1
- net LNA_IN: now also C7.1, U3.2 (LNA_IN); no longer C5.1
- new net: R7.2, R8.2, U4.8 (VBUS)
- new net: R12.1, U4.11 (SUSPEND)
- new net: R11.1, U4.9 (RST)
- new net: FPC1.1, U5.1
- new net: FPC1.10, U5.10
- new net: FPC1.11, U5.11
- new net: FPC1.12, U5.12
- new net: FPC1.2, U5.2
- new net: FPC1.3, U5.3
- new net: FPC1.4, U5.4
- new net: FPC1.5, U5.5
- new net: FPC1.6, U5.6
- new net: FPC1.7, U5.7
- new net: FPC1.8, U5.8
- new net: FPC1.9, U5.9
- new net: C4.1, R4.2, U3.9 (EN)
- new net: C5.1, C7.2, U2.1 (ANT)
- new net: R5.1, U3.18 (IO12)
- no-connect marks 16 -> 29
Other:
- moved on the sheet: C1, C3, D1, J1, J2, Q1, Q2, R1, R10, R13, R14, R15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

Commit message: update
Parts:
- added U6: SD-CARD, Uinika.Footprint:TF-SMD_SD-CARD, symbol Uinika:SD-CARD
- C10, C2, C4, C5, C6, C7, C8, C9: footprint Capacitor_SMD:C_0402_1005Metric -> Capacitor_SMD:C_0603_1608Metric
- FPC1: footprint kicad_lceda:FPC-SMD_12P-P0.50_FPC-05F-12PH20 -> Uinika.Footprint:FPC-SMD_12P-P0.50_FPC-05F-12PH20
- R1, R10, R11, R12, R13, R14, R15, R16, R2, R3, R4, R5, R6, R7, R8, R9: footprint Resistor_SMD:R_0402_1005Metric -> Resistor_SMD:R_0603_1608Metric
- SW1, SW2: footprint kicad_lceda:SW-SMD_L6.0-W3.3-LS8.0 -> Uinika.Footprint:SW-SMD_L6.0-W3.3-LS8.0
- U1: footprint Package_TO_SOT_SMD:SOT-223-3_TabPin2 -> Uinika.Footprint:SOT-23-3_L2.9-W1.6-P1.90-LS2.9-BL
- U2: footprint kicad_lceda:ANT-SMD_L5.0-W2.0 -> Uinika.Footprint:ANT-SMD_L5.0-W2.0
- U3: footprint kicad_lceda:QFN-48_L7.0-W7.0-P0.50-BL-EP5.4 -> Uinika.Footprint:QFN-48_L7.0-W7.0-P0.50-BL-EP5.4
- U4: footprint kicad_lceda:QFN-28_L5.0-W5.0-P0.50-TL-EP3.2-1 -> Uinika.Footprint:QFN-28_L5.0-W5.0-P0.50-TL-EP3.2-1
- U5: footprint kicad_lceda:FPC-SMD_12P-P1.00_XUNPU_FPC-1.0FX-12PWBH20 -> Uinika.Footprint:FPC-SMD_12P-P1.00_XUNPU_FPC-1.0FX-12PWBH20
- USB1: footprint kicad_lceda:USB-C-SMD_TYPEC-304J-BCP16 -> Uinika.Footprint:USB-C-SMD_TYPEC-304J-BCP16

Commit message: update
Parts:
- removed SW1, SW2: TD-1106SN-4.3H-160, Uinika.Footprint:SW-SMD_L6.0-W3.3-LS8.0, symbol Uinika:TD-1106SN-4.3H-160
- removed U6: SD-CARD, Uinika.Footprint:TF-SMD_SD-CARD, symbol Uinika:SD-CARD
- added C12: 10nF, Capacitor_SMD:C_0603_1608Metric, symbol Device:C
- added C13, C15, C9: 0.1uF, Capacitor_SMD:C_0603_1608Metric, symbol Device:C
- added C14: 2.2nF, Capacitor_SMD:C_0603_1608Metric, symbol Device:C
- added Card1: TF-02A_C2889261, Uinika.Footprint:TF-SMD_TF-02, symbol TF-SMD_TF-02:TF-02A_C2889261
- added Q1: AO3415AL, Uinika.Footprint:SOT-23-3_L2.9-W1.6-P1.90-LS2.9-BL, symbol kicad_lceda:AO3415AL
- added R19, R20, R21, R22, R6: 10k, Resistor_SMD:R_0603_1608Metric, symbol Device:R
- added R8: 1k, Resistor_SMD:R_0603_1608Metric, symbol Device:R
- added SW1, SW2: TD-1106SN-5.0H-160, Uinika.Footprint:SW-SMD_L6.0-W3.3-LS8.0-1, symbol Uinika:TD-1106SN-5.0H-160
- added U1: WS2812B-B, Uinika.Footprint:LED_WS2812B-B, symbol Uinika:WS2812B-B
- added U10: MPU6050-YJLTY, Uinika.Footprint:QFN-24_L4.0-W4.0-P0.50-BL-EP2.7, symbol Uinika:MPU6050-YJLTY
- added U4: BH1750FVI-TR, Uinika.Footprint:XDCR_BH1750FVI-TR, symbol Uinika:BH1750FVI-TR
- added U6: FPC-1.0FX-12PWBH20, Uinika.Footprint:FPC-SMD_12P-P1.00_XUNPU_FPC-1.0FX-12PWBH20, symbol Uinika:FPC-1.0FX-12PWBH20
- renumbered C9 to C10, C10 to C11, Q1 to Q2, Q2 to Q3, R8 to R10, R9 to R11, R10 to R12, R11 to R13, R12 to R14, R13 to R15, R14 to R16, R15 to R17, R16 to R18, R6 to R7, R7 to R9, U1 to U2, U2 to U3, U3 to U5, U4 to U7, U5 to U9
Connections:
- net DTR: no longer Q3.1 (E), R11.2
- net GND: now also C12.2, C13.1, C14.2, C15.2, C9.2, Card1.10 (GND), Card1.11 (GND), Card1.12 (GND), Card1.13 (GND), Card1.6 (VSS), Card1.9 (CD), SW1.1, SW2.1, U1.3 (VSS), U10.1 (CLKIN), U10.11 (FSYNC), U10.18 (GND), U10.9 (AD0), U4.2 (ADDR), U4.3 (GND), U6.1, U6.12, U6.2, U6.5, U6.6, U6.8
- net RTS: no longer Q2.1 (E), R12.2
- net at C2.2, R3.1: now also SW1.2
- net at C10.2, R7.1: now also SW2.2
- new net: R6.1, U4.5 (DVI)
- new net: Q2.1 (E), R12.2
- new net: C14.1, U10.20 (CPOUT)
- new net: Q1.1 (G), R8.1
- new net: C13.2, U10.10 (REGOUT)
- new net: Q1.3 (D), U6.3
- new net +3V3: C12.1, C15.1, C9.1, Card1.4 (VDD), Q1.2 (S), R19.2, R20.2, R21.2, R22.2, R6.2, U10.13 (VDD), U10.8 (VLOGIC), U4.1 (VCC), U6.4
- new net +5V: U1.1 (VDD)
- new net GPIO13/SD_MOSI: Card1.3 (CMD), R20.1
- new net GPIO14/SD_CLK: Card1.5 (CLK), R21.1
- new net GPIO15/SD_CS: Card1.2 (CD/DAT3), R22.1
- new net GPIO18/SCK: U6.9
- new net GPIO23/MOSI: U6.10
- new net GPIO26/SD_MISO: Card1.7 (DAT0), R19.1
- new net GPIO27/RGB_LED: U1.4 (DIN)
- new net GPIO2/DC: U6.7
- new net GPIO32/MPU_SDA/BH_SDA: U10.24 (SDA), U4.4 (SDA)
- new net GPIO33/MPU_SCL/BH_SCL: U10.23 (SCL), U4.6 (SCL)
- new net GPIO4/RES: U6.11
- new net GPIO5/LCD_BL: R8.2
- no-connect marks 29 -> 49
Other:
- note added: "ST7789 液晶屏"
- note added: "TF 存储卡"
- note added: "加速度传感器"
- moved on the sheet: C1, C10, C11, C2, C3, C4, C5, C6, C7, C8, D1, J1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

Commit message: update
Parts:
- renumbered U10 to U8
Connections:
- net +5V is gone; now on net EXT_5V: U1.1 (VDD)
- net GPIO18/SCK is gone; now on net IO18: U6.9
- net GPIO23/MOSI is gone; now on net IO23: U6.10
- net GPIO27/RGB_LED is gone; now on net IO27: U1.4 (DIN)
- net GPIO2/DC is gone; now on net IO2: U6.7
- net GPIO32/MPU_SDA/BH_SDA is gone; now on net IO32: U4.4 (SDA), U8.24 (SDA)
- net GPIO33/MPU_SCL/BH_SCL is gone; now on net IO33: U4.6 (SCL), U8.23 (SCL)
- net GPIO4/RES is gone; now on net IO4: U6.11
- net GPIO5/LCD_BL is gone; now on net IO5: R8.2
- net +3V3: no longer C12.1, C15.1, C9.1, Q1.2 (S), R6.2, U4.1 (VCC), U6.4, U8.13 (VDD), U8.8 (VLOGIC)
- net VDD33: now also C12.1, C15.1, C9.1, Q1.2 (S), R6.2, U4.1 (VCC), U6.4, U8.13 (VDD), U8.8 (VLOGIC)
Other:
- note added: "WS2812B RGB LED"
- moved on the sheet: C1, C10, C11, C12, C13, C14, C15, C2, C3, C4, C5, C6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

Commit message: update
Parts:
- added C16: 10uF, Capacitor_SMD:C_0603_1608Metric, symbol Device:C
- added C17: 0.1uF, Capacitor_SMD:C_0603_1608Metric, symbol Device:C
- added C18: 10nF, Capacitor_SMD:C_0603_1608Metric, symbol Device:C
- added J1: Conn_01x02_Male, Connector_PinHeader_2.54mm:PinHeader_1x02_P2.54mm_Vertical, symbol Connector:Conn_01x02_Male
- added J2: Conn_01x04_Male, Connector_PinHeader_2.54mm:PinHeader_1x04_P2.54mm_Vertical, symbol Connector:Conn_01x04_Male
- added U9: LP2992IM5-3.3, Uinika.Footprint:SOT95P280X145-5N, symbol Uinika:LP2992IM5-3.3
- added USB2: TYPEC-304J-BCP16, Uinika.Footprint:USB-C-SMD_TYPEC-304J-BCP16, symbol Uinika:TYPEC-304J-BCP16
- renumbered C2 to C1, C3 to C10, C4 to C2, C5 to C3, C6 to C4, C7 to C5, C8 to C6, C1 to C7, C9 to C8, C10 to C9, J1 to J3, J2 to J4, R2 to R1, R16 to R10, R17 to R11, R18 to R12, R9 to R13, R10 to R14, R13 to R15, R14 to R16, R11 to R17, R12 to R18, R3 to R2, R4 to R3, R5 to R4, R6 to R5, R1 to R6, R15 to R9, U9 to U10, U3 to U2, U4 to U3, U5 to U4, U2 to U5
Connections:
- net +3V3: now also C16.2, C17.2, J2.1 (Pin_1), U9.5 (VOUT)
- net EXT_5V: now also C7.1, R6.1, U5.3 (VI)
- net GND: now also C16.1, C17.1, C18.2, J1.1 (Pin_1), J2.2 (Pin_2), U9.2 (GND), USB2.13 (GND), USB2.14 (GND), USB2.15 (GND), USB2.16 (GND), USB2.A1B12 (GND), USB2.B1A12 (GND)
- net VDD33: now also J1.2 (Pin_2)
- new net: C18.1, U9.4 (BYPASS)
- new net USB_5V: U9.1 (VIN), U9.3 (ON/~{OFF}), USB2.A4B9 (VBUS), USB2.B4A9 (VBUS)
- new net USB_CON+: J2.3 (Pin_3), USB2.A6 (DP1), USB2.B6 (DP2)
- new net USB_CON-: J2.4 (Pin_4), USB2.A7 (DN1), USB2.B7 (DN2)
- no-connect marks 49 -> 53
Other:
- note added: "AMS1117-3.3 电源"
- note removed: "电源"
- moved on the sheet: C10, C11, C12, C13, C14, C15, C7, C8, Card1, D1, FPC1, J3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
