File: Hardware/Egret.kicad_sch (KiCad schematic)
At the start: 65 parts, among them J1 Conn_01x02_Male, J2 Conn_01x04_Male, J3 Conn_01x20_Male, J4 Conn_01x20_Male, Q1 AO3415AL, Q2 S8050, Q3 S8050, SW1 TD-1106SN-5.0H-160, SW2 TD-1106SN-5.0H-160, U1 WS2812B-B, U10 FPC-1.0FX-12PWBH20, U2 AN2051-245_2.4G, U3 BH1750FVI-TR, U4 ESP32--PICO--D4, U5 AMS1117-3.3, U6 FPC-1.0FX-12PWBH20, U7 CP2102-GMR-YJLTY, U8 MPU6050-YJLTY, U9 LP2992IM5-3.3

Commit message: update
Other:
- note added: "LP2992 线性稳压器"
- moved on the sheet: C16, C17, C18, J2, U9, USB2

Commit message: update
Parts:
- removed Card1: TF-02A_C2889261, Uinika.Footprint:TF-SMD_TF-02, symbol TF-SMD_TF-02:TF-02A_C2889261
- removed Q1: AO3415AL, Uinika.Footprint:SOT-23-3_L2.9-W1.6-P1.90-LS2.9-BL, symbol kicad_lceda:AO3415AL
- removed R13: 47.5K(1%), Resistor_SMD:R_0603_1608Metric, symbol Device:R
- removed U7: CP2102-GMR-YJLTY, Uinika.Footprint:QFN-28_L5.0-W5.0-P0.50-TL-EP3.2-1, symbol Uinika:CP2102-GMR-YJLTY
- added Card1: TF-02A_C2889261, kicad_lceda:TF-SMD_TF-02, symbol Uinika:TF-02A_C2889261
- added Q1: AO3415AL, kicad_lceda:SOT-23-3_L2.9-W1.6-P1.90-LS2.9-BL, symbol Uinika:AO3415AL
- added R9: 47.5K(1%), Resistor_SMD:R_0603_1608Metric, symbol Device:R
- added U7: CP2102N-A02-GQFN28, kicad_lceda:QFN-28_L5.0-W5.0-P0.50-TL-EP3.3, symbol Uinika:CP2102N-A02-GQFN28
- FPC1: footprint Uinika.Footprint:FPC-SMD_12P-P0.50_FPC-05F-12PH20 -> kicad_lceda:FPC-SMD_12P-P0.50_FPC-05F-12PH20
- U10, U6: footprint Uinika.Footprint:FPC-SMD_12P-P1.00_XUNPU_FPC-1.0FX-12PWBH20 -> kicad_lceda:FPC-SMD_12P-P1.00_XUNPU_FPC-1.0FX-12PWBH20
- U4: footprint Uinika.Footprint:QFN-48_L7.0-W7.0-P0.50-BL-EP5.4 -> kicad_lceda:QFN-48_L7.0-W7.0-P0.50-BL-EP5.4
- U8: footprint Uinika.Footprint:QFN-24_L4.0-W4.0-P0.50-BL-EP2.7 -> kicad_lceda:QFN-24_L4.0-W4.0-P0.50-BL-EP2.7
- USB1, USB2: footprint Uinika.Footprint:USB-C-SMD_TYPEC-304J-BCP16 -> kicad_lceda:USB-C-SMD_TYPEC-304J-BCP16
- renumbered R9 to R10, R10 to R11, R11 to R12, R12 to R13
Connections:
- net CTS: now also U7.23 (CTS)
- net DTR: now also Q3.1 (E), R17.2, U7.28 (DTR)
- net GND: now also Card1.1 (DAT2), Card1.10 (GND), Card1.11 (GND), Card1.12 (GND), Card1.13 (GND), Card1.4 (VDD), R9.1, U7.29 (EP), U7.3 (GND)
- net GPIO13/SD_MOSI: now also Card1.7 (DAT0)
- net GPIO14/SD_CLK: now also Card1.5 (CLK)
- net GPIO15/SD_CS: now also Card1.8 (DAT1)
- net GPIO26/SD_MISO: now also Card1.3 (CMD)
- net RTS: now also Q2.1 (E), R18.2, U7.24 (RTS)
- net RXD: now also U7.25 (RXD)
- net TXD: now also U7.26 (TXD)
- net USB_DN: now also U7.5 (D-)
- net USB_DP: now also U7.4 (D+)
- net VDD33: now also R19.2, R20.2, R21.2, R22.2, Card1.6 (VSS), Q1.2 (S), U7.6 (VDD), U7.7 (VREGIN)
- net at R14.2: now also R9.2, U7.8 (VBUS)
- net at R16.1: now also U7.11 (SUSPENDb)
- net at R15.1: now also U7.9 (RSTb)
- net at R8.1: now also Q1.1 (G)
- net at U6.3: now also Q1.3 (D)
- net +3V3: no longer names the net of C16.2, C17.2, J2.1 (Pin_1), U9.5 (VOUT)
- net +3V3: no longer R19.2, R20.2, R21.2, R22.2

Commit message: update
Parts:
- Card1: footprint kicad_lceda:TF-SMD_TF-02 -> Uinika.Footprint:TF-SMD_TF-02
- FPC1: footprint kicad_lceda:FPC-SMD_12P-P0.50_FPC-05F-12PH20 -> Uinika.Footprint:FPC-SMD_12P-P0.50_FPC-05F-12PH20
- Q1: footprint kicad_lceda:SOT-23-3_L2.9-W1.6-P1.90-LS2.9-BL -> Uinika.Footprint:SOT-23-3_L2.9-W1.6-P1.90-LS2.9-BL
- U10, U6: footprint kicad_lceda:FPC-SMD_12P-P1.00_XUNPU_FPC-1.0FX-12PWBH20 -> Uinika.Footprint:FPC-SMD_12P-P1.00_XUNPU_FPC-1.0FX-12PWBH20
- U4: footprint kicad_lceda:QFN-48_L7.0-W7.0-P0.50-BL-EP5.4 -> Uinika.Footprint:QFN-48_L7.0-W7.0-P0.50-BL-EP5.4
- U7: footprint kicad_lceda:QFN-28_L5.0-W5.0-P0.50-TL-EP3.3 -> Uinika.Footprint:QFN-28_L5.0-W5.0-P0.50-TL-EP3.3
- U8: footprint kicad_lceda:QFN-24_L4.0-W4.0-P0.50-BL-EP2.7 -> Uinika.Footprint:QFN-24_L4.0-W4.0-P0.50-BL-EP2.7
- USB1, USB2: footprint kicad_lceda:USB-C-SMD_TYPEC-304J-BCP16 -> Uinika.Footprint:USB-C-SMD_TYPEC-304J-BCP16
Changed lines of the file:
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@@
     (property "Reference" "USB2" (id 0) (at 363.22 29.972 0))
     (property "Value" "TYPEC-304J-BCP16" (id 1) (at 363.22 32.512 0))
-    (property "Footprint" "kicad_lceda:USB-C-SMD_TYPEC-304J-BCP16" (id 2) (at 361.95 66.294 0)
+    (property "Footprint" "Uinika.Footprint:USB-C-SMD_TYPEC-304J-BCP16" (id 2) (at 361.95 66.294 0)
       (effects (font (size 1.27 1.27)) hide)
     )
@@
     (property "Reference" "USB1" (id 0) (at 83.566 33.782 0))
     (property "Value" "TYPEC-304J-BCP16" (id 1) (at 83.566 73.66 0))
-    (property "Footprint" "kicad_lceda:USB-C-SMD_TYPEC-304J-BCP16" (id 2) (at 82.042 68.326 0)
+    (property "Footprint" "Uinika.Footprint:USB-C-SMD_TYPEC-304J-BCP16" (id 2) (at 82.042 68.326 0)
       (effects (font (size 1.27 1.27)) hide)
     )
@@
     (property "Reference" "Card1" (id 0) (at 511.048 150.368 0))
     (property "Value" "TF-02A_C2889261" (id 1) (at 511.048 152.908 0))
-    (property "Footprint" "kicad_lceda:TF-SMD_TF-02" (id 2) (at 511.048 158.496 0)
+    (property "Footprint" "Uinika.Footprint:TF-SMD_TF-02" (id 2) (at 511.048 158.496 0)
       (effects (font (size 1.27 1.27)) hide)
     )
@@
     (property "Reference" "U4" (id 0) (at 162.306 205.74 0))
     (property "Value" "ESP32--PICO--D4" (id 1) (at 162.306 208.28 0))
-    (property "Footprint" "kicad_lceda:QFN-48_L7.0-W7.0-P0.50-BL-EP5.4" (id 2) (at 162.306 136.398 0)
+    (property "Footprint" "Uinika.Footprint:QFN-48_L7.0-W7.0-P0.50-BL-EP5.4" (id 2) (at 162.306 136.398 0)
       (effects (font (size 1.27 1.27)) hide)
     )
@@
       (effects (font (size 1.27 1.27)) (justify left))
     )
-    (property "Footprint" "kicad_lceda:FPC-SMD_12P-P0.50_FPC-05F-12PH20" (id 2) (at 485.14 320.1924 0)
+    (property "Footprint" "Uinika.Footprint:FPC-SMD_12P-P0.50_FPC-05F-12PH20" (id 2) (at 485.14 320.1924 0)
       (effects (font (size 1.27 1.27)) hide)
     )
@@
       (effects (font (size 1.27 1.27)) (justify left))
     )
-    (property "Footprint" "kicad_lceda:FPC-SMD_12P-P1.00_XUNPU_FPC-1.0FX-12PWBH20" (id 2) (at 527.05 320.1924 0)
+    (property "Footprint" "Uinika.Footprint:FPC-SMD_12P-P1.00_XUNPU_FPC-1.0FX-12PWBH20" (id 2) (at 527.05 320.1924 0)
       (effects (font (size 1.27 1.27)) hide)
     )
@@
       (effects (font (size 1.27 1.27)) (justify left))
     )
-    (property "Footprint" "kicad_lceda:QFN-24_L4.0-W4.0-P0.50-BL-EP2.7" (id 2) (at 376.428 322.2244 0)
+    (property "Footprint" "Uinika.Footprint:QFN-24_L4.0-W4.0-P0.50-BL-EP2.7" (id 2) (at 376.428 322.2244 0)
       (effects (font (size 1.27 1.27)) hide)
     )
@@
       (effects (font (size 1.27 1.27)) (justify left))
     )
-    (property "Footprint" "kicad_lceda:SOT-23-3_L2.9-W1.6-P1.90-LS2.9-BL" (id 2) (at 220.218 335.534 0)
+    (property "Footprint" "Uinika.Footprint:SOT-23-3_L2.9-W1.6-P1.90-LS2.9-BL" (id 2) (at 220.218 335.534 0)
       (effects (font (size 1.27 1.27)) hide)
     )
@@
     (property "Reference" "U7" (id 0) (at 371.856 129.286 0))
     (property "Value" "CP2102N-A02-GQFN28" (id 1) (at 371.856 131.826 0))
-    (property "Footprint" "kicad_lceda:QFN-28_L5.0-W5.0-P0.50-TL-EP3.3" (id 2) (at 371.856 136.6266 0)
+    (property "Footprint" "Uinika.Footprint:QFN-28_L5.0-W5.0-P0.50-TL-EP3.3" (id 2) (at 371.856 136.6266 0)
       (effects (font (size 1.27 1.27)) hide)
     )
@@
       (effects (font (size 1.27 1.27)) (justify left))
     )
-    (property "Footprint" "kicad_lceda:FPC-SMD_12P-P1.00_XUNPU_FPC-1.0FX-12PWBH20" (id 2) (at 280.67 325.0184 0)
+    (property "Footprint" "Uinika.Footprint:FPC-SMD_12P-P1.00_XUNPU_FPC-1.0FX-12PWBH20" (id 2) (at 280.67 325.0184 0)
       (effects (font (size 1.27 1.27)) hide)
     )
@@
     )
     (path "/3afcb223-47b2-471c-b033-efe4cf031aa7"
-      (reference "Card1") (unit 1) (value "TF-02A_C2889261") (footprint "kicad_lceda:TF-SMD_TF-02")
+      (reference "Card1") (unit 1) (value "TF-02A_C2889261") (footprint "Uinika.Footprint:TF-SMD_TF-02")
     )
     (path "/432c7922-80d6-44fb-bad2-9be5e483decf"
@@
     )
     (path "/4b170995-b1c2-4f50-b1cc-679a8a17ed4c"
-      (reference "FPC1") (unit 1) (value "FPC-05F-12PH20") (footprint "kicad_lceda:FPC-SMD_12P-P0.50_FPC-05F-12PH20")
+      (reference "FPC1") (unit 1) (value "FPC-05F-12PH20") (footprint "Uinika.Footprint:FPC-SMD_12P-P0.50_FPC-05F-12PH20")
     )
     (path "/d96f9893-c62f-4f43-b5ae-b0c08e7930fa"
@@
     )
     (path "/f559a1cb-114f-43d6-9a93-35849bfdfb8e"
-      (reference "Q1") (unit 1) (value "AO3415AL") (footprint "kicad_lceda:SOT-23-3_L2.9-W1.6-P1.90-LS2.9-BL")
+      (reference "Q1") (unit 1) (value "AO3415AL") (footprint "Uinika.Footprint:SOT-23-3_L2.9-W1.6-P1.90-LS2.9-BL")
     )
     (path "/cb03a087-40d7-41e9-917a-781abe0f15aa"
@@
     )
     (path "/480bab45-8f57-4218-ba03-9a440e4bc782"
-      (reference "U4") (unit 1) (value "ESP32--PICO--D4") (footprint "kicad_lceda:QFN-48_L7.0-W7.0-P0.50-BL-EP5.4")
+      (reference "U4") (unit 1) (value "ESP32--PICO--D4") (footprint "Uinika.Footprint:QFN-48_L7.0-W7.0-P0.50-BL-EP5.4")
     )
     (path "/54035f82-7250-4b57-8dcd-38ee49cb329d"
@@
     )
     (path "/fd4d85a6-0a5a-451a-b143-ec755ed9eb0e"
-      (reference "U6") (unit 1) (value "FPC-1.0FX-12PWBH20") (footprint "kicad_lceda:FPC-SMD_12P-P1.00_XUNPU_FPC-1.0FX-12PWBH20")
+      (reference "U6") (unit 1) (value "FPC-1.0FX-12PWBH20") (footprint "Uinika.Footprint:FPC-SMD_12P-P1.00_XUNPU_FPC-1.0FX-12PWBH20")
     )
     (path "/f609a517-7771-41e1-b842-051a4a7dbcb3"
-      (reference "U7") (unit 1) (value "CP2102N-A02-GQFN28") (footprint "kicad_lceda:QFN-28_L5.0-W5.0-P0.50-TL-EP3.3")
+      (reference "U7") (unit 1) (value "CP2102N-A02-GQFN28") (footprint "Uinika.Footprint:QFN-28_L5.0-W5.0-P0.50-TL-EP3.3")
     )
     (path "/a6426d11-8451-4e3b-8d15-afb778a9f71c"
-      (reference "U8") (unit 1) (value "MPU6050-YJLTY") (footprint "kicad_lceda:QFN-24_L4.0-W4.0-P0.50-BL-EP2.7")
+      (reference "U8") (unit 1) (value "MPU6050-YJLTY") (footprint "Uinika.Footprint:QFN-24_L4.0-W4.0-P0.50-BL-EP2.7")
     )
     (path "/cb903857-b34d-4db5-8932-008ede2a3952"
@@
     )
     (path "/739fbc58-5133-4e40-b700-18a058a58ad7"
-      (reference "U10") (unit 1) (value "FPC-1.0FX-12PWBH20") (footprint "kicad_lceda:FPC-SMD_12P-P1.00_XUNPU_FPC-1.0FX-12PWBH20")
+      (reference "U10") (unit 1) (value "FPC-1.0FX-12PWBH20") (footprint "Uinika.Footprint:FPC-SMD_12P-P1.00_XUNPU_FPC-1.0FX-12PWBH20")
     )
     (path "/2ee5bc88-a7a5-48cd-9011-35833e008869"
-      (reference "USB1") (unit 1) (value "TYPEC-304J-BCP16") (footprint "kicad_lceda:USB-C-SMD_TYPEC-304J-BCP16")
+      (reference "USB1") (unit 1) (value "TYPEC-304J-BCP16") (footprint "Uinika.Footprint:USB-C-SMD_TYPEC-304J-BCP16")
     )
     (path "/2b5867a7-143c-4827-9ce9-514bd547d48c"
-      (reference "USB2") (unit 1) (value "TYPEC-304J-BCP16") (footprint "kicad_lceda:USB-C-SMD_TYPEC-304J-BCP16")
-    )
-  )
+      (reference "USB2") (unit 1) (value "TYPEC-304J-BCP16") (footprint "Uinika.Footprint:USB-C-SMD_TYPEC-304J-BCP16")
+    )
+  )

Commit message: update
Connections:
- net GPIO13/SD_MOSI is gone; now on net IO13: Card1.7 (DAT0), R20.1
- net GPIO14/SD_CLK is gone; now on net IO14: Card1.5 (CLK), R21.1
- net GPIO15/SD_CS is gone; now on net IO15: Card1.8 (DAT1), R22.1
- net GPIO26/SD_MISO is gone; now on net IO26: Card1.3 (CMD), R19.1
- net at FPC1.1: now also U10.12; no longer U10.1
- net at FPC1.10: now also U10.3; no longer U10.10
- net at FPC1.11: now also U10.2; no longer U10.11
- net at FPC1.12: now also U10.1; no longer U10.12
- net at FPC1.2: now also U10.11; no longer U10.2
- net at FPC1.3: now also U10.10; no longer U10.3
- net at FPC1.4: now also U10.9; no longer U10.4
- net at FPC1.5: now also U10.8; no longer U10.5
- net at FPC1.6: now also U10.7; no longer U10.6
- net at FPC1.7: now also U10.6; no longer U10.7
- net at FPC1.8: now also U10.5; no longer U10.8
- net at FPC1.9: now also U10.4; no longer U10.9
Changed lines of the file:
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@@
     (effects (font (size 1.27 1.27)) (justify right bottom))
   )
-  (label "GPIO15{slash}SD_CS" (at 486.664 176.276 180)
+  (label "IO15" (at 486.664 176.276 180)
     (effects (font (size 1.27 1.27)) (justify right bottom))
   )
@@
     (effects (font (size 1.27 1.27)) (justify right bottom))
   )
-  (label "GPIO26{slash}SD_MISO" (at 494.03 163.576 180)
+  (label "IO26" (at 494.03 163.576 180)
     (effects (font (size 1.27 1.27)) (justify right bottom))
   )
@@
     (effects (font (size 1.27 1.27)) (justify right bottom))
   )
-  (label "GPIO15{slash}SD_CS" (at 497.332 135.89 180)
+  (label "IO15" (at 497.332 135.89 180)
     (effects (font (size 1.27 1.27)) (justify right bottom))
   )
@@
     (effects (font (size 1.27 1.27)) (justify left bottom))
   )
-  (label "GPIO13{slash}SD_MOSI" (at 497.332 124.46 180)
+  (label "IO13" (at 497.332 124.46 180)
     (effects (font (size 1.27 1.27)) (justify right bottom))
   )
@@
     (effects (font (size 1.27 1.27)) (justify right bottom))
   )
-  (label "GPIO13{slash}SD_MOSI" (at 486.664 173.736 180)
+  (label "IO13" (at 486.664 173.736 180)
     (effects (font (size 1.27 1.27)) (justify right bottom))
   )
@@
     (effects (font (size 1.27 1.27)) (justify right bottom))
   )
-  (label "GPIO26{slash}SD_MISO" (at 497.332 118.618 180)
+  (label "IO26" (at 497.332 118.618 180)
     (effects (font (size 1.27 1.27)) (justify right bottom))
   )
@@
     (effects (font (size 1.27 1.27)) (justify left bottom))
   )
-  (label "GPIO14{slash}SD_CLK" (at 497.332 130.048 180)
+  (label "IO14" (at 497.332 130.048 180)
     (effects (font (size 1.27 1.27)) (justify right bottom))
   )
@@
     (effects (font (size 1.27 1.27)) (justify right bottom))
   )
-  (label "GPIO14{slash}SD_CLK" (at 485.902 168.656 180)
+  (label "IO14" (at 485.902 168.656 180)
     (effects (font (size 1.27 1.27)) (justify right bottom))
   )
@@
   (symbol (lib_id "power:GND") (at 532.13 178.816 90) (unit 1)
     (in_bom yes) (on_board yes) (fields_autoplaced)
-    (property "Reference" "#PWR047" (id 0) (at 538.48 178.816 0)
+    (property "Reference" "#PWR044" (id 0) (at 538.48 178.816 0)
       (effects (font (size 1.27 1.27)) hide)
     )
@@
   (symbol (lib_id "power:GND") (at 498.348 158.496 270) (unit 1)
     (in_bom yes) (on_board yes) (fields_autoplaced)
-    (property "Reference" "#PWR042" (id 0) (at 491.998 158.496 0)
+    (property "Reference" "#PWR040" (id 0) (at 491.998 158.496 0)
       (effects (font (size 1.27 1.27)) hide)
     )
@@
   (symbol (lib_id "power:GND") (at 532.638 161.036 90) (unit 1)
     (in_bom yes) (on_board yes) (fields_autoplaced)
-    (property "Reference" "#PWR048" (id 0) (at 538.988 161.036 0)
+    (property "Reference" "#PWR045" (id 0) (at 538.988 161.036 0)
       (effects (font (size 1.27 1.27)) hide)
     )
@@
   (symbol (lib_id "power:GND") (at 494.03 166.116 270) (unit 1)
     (in_bom yes) (on_board yes)
-    (property "Reference" "#PWR040" (id 0) (at 487.68 166.116 0)
+    (property "Reference" "#PWR039" (id 0) (at 487.68 166.116 0)
       (effects (font (size 1.27 1.27)) hide)
     )
@@
   (symbol (lib_id "power:GND") (at 525.018 176.276 90) (unit 1)
     (in_bom yes) (on_board yes) (fields_autoplaced)
-    (property "Reference" "#PWR044" (id 0) (at 531.368 176.276 0)
+    (property "Reference" "#PWR042" (id 0) (at 531.368 176.276 0)
       (effects (font (size 1.27 1.27)) hide)
     )
@@
     (pin "1")
   )
-  (symbol (lib_name "FPC-1.0FX-12PWBH20_1") (lib_id "Uinika:FPC-1.0FX-12PWBH20") (at 527.05 337.312 0) (unit 1)
-    (in_bom yes) (on_board yes) (fields_autoplaced)
-    (property "Reference" "U10" (id 0) (at 533.146 336.0419 0)
-      (effects (font (size 1.27 1.27)) (justify left))
-    )
-    (property "Value" "FPC-1.0FX-12PWBH20" (id 1) (at 533.146 338.5819 0)
-      (effects (font (size 1.27 1.27)) (justify left))
-    )
-    (property "Footprint" "Uinika.Footprint:FPC-SMD_12P-P1.00_XUNPU_FPC-1.0FX-12PWBH20" (id 2) (at 527.05 320.1924 0)
-      (effects (font (size 1.27 1.27)) hide)
-    )
-    (property "Datasheet" "" (id 3) (at 527.05 325.2724 0)
-      (effects (font (size 1.27 1.27)) hide)
-    )
-    (property "SuppliersPartNumber" "C3446098" (id 4) (at 527.05 330.3778 0)
-      (effects (font (size 1.27 1.27)) hide)
-    )
-    (property "uuid" "std:b32b34129bde432394d92692ef7ead04" (id 5) (at 527.05 330.3778 0)
+  (symbol (lib_name "FPC-1.0FX-12PWBH20_1") (lib_id "Uinika:FPC-1.0FX-12PWBH20") (at 527.05 337.312 0) (mirror x) (unit 1)
+    (in_bom yes) (on_board yes) (fields_autoplaced)
+    (property "Reference" "U10" (id 0) (at 533.4 336.0419 0)
+      (effects (font (size 1.27 1.27)) (justify left))
+    )
+    (property "Value" "FPC-1.0FX-12PWBH20" (id 1) (at 533.4 338.5819 0)
+      (effects (font (size 1.27 1.27)) (justify left))
+    )
+    (property "Footprint" "Uinika.Footprint:FPC-SMD_12P-P1.00_XUNPU_FPC-1.0FX-12PWBH20" (id 2) (at 527.05 354.4316 0)
+      (effects (font (size 1.27 1.27)) hide)
+    )
+    (property "Datasheet" "" (id 3) (at 527.05 349.3516 0)
+      (effects (font (size 1.27 1.27)) hide)
+    )
+    (property "SuppliersPartNumber" "C3446098" (id 4) (at 527.05 344.2462 0)
+      (effects (font (size 1.27 1.27)) hide)
+    )
+    (property "uuid" "std:b32b34129bde432394d92692ef7ead04" (id 5) (at 527.05 344.2462 0)
       (effects (font (size 1.27 1.27)) hide)
     )
@@
   (symbol (lib_id "power:GND") (at 528.066 40.386 0) (mirror x) (unit 1)
     (in_bom yes) (on_board yes) (fields_autoplaced)
-    (property "Reference" "#PWR045" (id 0) (at 528.066 34.036 0)
+    (property "Reference" "#PWR043" (id 0) (at 528.066 34.036 0)
       (effects (font (size 1.27 1.27)) hide)
     )
@@
   (symbol (lib_id "power:GND") (at 524.764 158.496 90) (unit 1)
     (in_bom yes) (on_board yes) (fields_autoplaced)
-    (property "Reference" "#PWR043" (id 0) (at 531.114 158.496 0)
+    (property "Reference" "#PWR041" (id 0) (at 531.114 158.496 0)
       (effects (font (size 1.27 1.27)) hide)
     )
@@
   (symbol (lib_id "power:GND") (at 477.266 63.246 270) (mirror x) (unit 1)
     (in_bom yes) (on_board yes) (fields_autoplaced)
-    (property "Reference" "#PWR039" (id 0) (at 470.916 63.246 0)
+    (property "Reference" "#PWR038" (id 0) (at 470.916 63.246 0)
       (effects (font (size 1.27 1.27)) hide)
     )
@@
     )
     (path "/fa850820-be88-4359-ad9f-47a8136c05a3"
+      (reference "#PWR038") (unit 1) (value "GND") (footprint "")
+    )
+    (path "/46db4203-03bb-47e8-a360-1af7d860d18d"
       (reference "#PWR039") (unit 1) (value "GND") (footprint "")
     )
-    (path "/46db4203-03bb-47e8-a360-1af7d860d18d"
+    (path "/1851ce90-15e6-4147-b28d-9d63c360bd01"
       (reference "#PWR040") (unit 1) (value "GND") (footprint "")
     )
-    (path "/1851ce90-15e6-4147-b28d-9d63c360bd01"
+    (path "/bd877408-3629-4ffd-8511-3752b1f7e5a0"
+      (reference "#PWR041") (unit 1) (value "GND") (footprint "")
+    )
+    (path "/631110fa-fe51-496e-996a-c518674b7d3c"
       (reference "#PWR042") (unit 1) (value "GND") (footprint "")
     )
-    (path "/bd877408-3629-4ffd-8511-3752b1f7e5a0"
+    (path "/aacf981a-87c7-4619-94b8-44ece360e140"
       (reference "#PWR043") (unit 1) (value "GND") (footprint "")
     )
-    (path "/631110fa-fe51-496e-996a-c518674b7d3c"
+    (path "/0495ef3c-2227-42f5-b3ac-bbb6656c75e6"
       (reference "#PWR044") (unit 1) (value "GND") (footprint "")
     )
-    (path "/aacf981a-87c7-4619-94b8-44ece360e140"
+    (path "/4491e308-ebe7-43b8-bd1b-d0ab47bfda7e"
       (reference "#PWR045") (unit 1) (value "GND") (footprint "")
     )
-    (path "/0495ef3c-2227-42f5-b3ac-bbb6656c75e6"
-      (reference "#PWR047") (unit 1) (value "GND") (footprint "")
-    )
-    (path "/4491e308-ebe7-43b8-bd1b-d0ab47bfda7e"
-      (reference "#PWR048") (unit 1) (value "GND") (footprint "")
-    )
     (path "/774cfaad-fc20-49a5-ad77-46609df84de6"

Commit message: update
Parts:
- removed C16: 10uF, Capacitor_SMD:C_0603_1608Metric, symbol Device:C
- removed C17: 0.1uF, Capacitor_SMD:C_0603_1608Metric, symbol Device:C
- removed C18: 10nF, Capacitor_SMD:C_0603_1608Metric, symbol Device:C
- removed FPC1: FPC-05F-12PH20, Uinika.Footprint:FPC-SMD_12P-P0.50_FPC-05F-12PH20, symbol Uinika:FPC-05F-12PH20
- removed J2: Conn_01x04_Male, Connector_PinHeader_2.54mm:PinHeader_1x04_P2.54mm_Vertical, symbol Connector:Conn_01x04_Male
- removed J3, J4: Conn_01x20_Male, Connector_PinHeader_2.54mm:PinHeader_1x20_P2.54mm_Vertical, symbol Connector:Conn_01x20_Male
- removed U10, U6: FPC-1.0FX-12PWBH20, Uinika.Footprint:FPC-SMD_12P-P1.00_XUNPU_FPC-1.0FX-12PWBH20, symbol Uinika:FPC-1.0FX-12PWBH20
- removed U9: LP2992IM5-3.3, Uinika.Footprint:SOT95P280X145-5N, symbol Uinika:LP2992IM5-3.3
- removed USB2: TYPEC-304J-BCP16, Uinika.Footprint:USB-C-SMD_TYPEC-304J-BCP16, symbol Uinika:TYPEC-304J-BCP16
- added U10: ST7789_FPC_PAD, symbol Uinika:ST7789_FPC_PAD
- added U8, U9: FPC-SMD_8P-P0.5, Uinika.Footprint:FPC-SMD_8P-P0.5_C9900011879, symbol Uinika:FPC-SMD_8P-P0.5
- renumbered C9 to C10, C14 to C11, C15 to C12, C10 to C13, C8 to C14, C11 to C15, C12 to C7, C7 to C8, C13 to C9, Q2 to Q1, Q3 to Q2, Q1 to Q3, R12 to R10, R13 to R11, R14 to R12, R15 to R13, R16 to R14, R5 to R15, R17 to R16, R18 to R17, R8 to R18, R6 to R5, R7 to R6, R9 to R7, R10 to R8, R11 to R9, U4 to U3, U8 to U4, U3 to U6
Connections:
- net VDD33 is gone; now on net EXT_5V: C12.1, C13.1, C14.1, C15.1, C7.1, Card1.6 (VSS), J1.2 (Pin_2), Q3.2 (S), R1.2, R13.2, R15.2, R19.2, R20.2, R21.2, R22.2, R4.2, U4.13 (VDD), U4.8 (VLOGIC), U5.2 (VO), U6.1 (VCC), U7.6 (VDD), U7.7 (VREGIN)
- net EXT_5V: now also U10.4 (VDD), U8.7, U8.8, U9.1, U9.2
- net GND: now also U10.1 (GND), U10.12 (GND), U10.2 (LEDK), U10.5 (GND), U10.6 (GND), U10.8 (CS), U8.6, U9.3
- net IO18: now also U10.9 (SCL), U8.4, U9.5
- net IO2: now also U10.7 (DC), U8.5, U9.4
- net IO23: now also U10.10 (SDA), U8.3, U9.6
- net IO4: now also U10.11 (RES), U8.2, U9.7
- net IO5: now also U8.1, U9.8
- net at Q3.3 (D): now also U10.3 (LEDA)
- no-connect marks 53 -> 47
Other:
- note added: "BH1750 光线传感器"
- note added: "MP6050 加速度传感器"
- note added: "ST7789 液晶显示屏"
- note removed: "LP2992 线性稳压器"
- note removed: "ST7789 液晶屏"
- note removed: "加速度传感器"
- note removed: "排针"
- moved on the sheet: C1, C10, C11, C12, C14, C15, C2, C3, C4, C5, C6, C7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

Commit message: update
Parts:
- L1: footprint Inductor_SMD:L_0402_1005Metric -> Inductor_SMD:L_0603_1608Metric
- U10: footprint (none) -> Uinika.Footprint:ST7789-FPC-PAD
Connections:
- net EXT_5V: no longer C12.1, C13.1, C14.1, C15.1, C7.1, Card1.6 (VSS), J1.2 (Pin_2), Q3.2 (S), R1.2, R13.2, R15.2, R19.2, R20.2, R21.2, R22.2, R4.2, U10.4 (VDD), U4.13 (VDD), U4.8 (VLOGIC), U5.2 (VO), U6.1 (VCC), U7.6 (VDD), U7.7 (VREGIN), U8.7, U8.8, U9.1, U9.2
- new net VDD33: C12.1, C13.1, C14.1, C15.1, C7.1, Card1.6 (VSS), J1.2 (Pin_2), Q3.2 (S), R1.2, R13.2, R15.2, R19.2, R20.2, R21.2, R22.2, R4.2, U10.4 (VDD), U4.13 (VDD), U4.8 (VLOGIC), U5.2 (VO), U6.1 (VCC), U7.6 (VDD), U7.7 (VREGIN), U8.7, U8.8, U9.1, U9.2
