File: Hardware/Egret.kicad_sch (KiCad schematic)
At the start: 57 parts, among them J1 Conn_01x02_Male, Q1 S8050, Q2 S8050, Q3 AO3415AL, SW1 TD-1106SN-5.0H-160, SW2 TD-1106SN-5.0H-160, U1 WS2812B-B, U10 ST7789_FPC_PAD, U2 AN2051-245_2.4G, U3 ESP32--PICO--D4, U4 MPU6050-YJLTY, U5 AMS1117-3.3, U6 BH1750FVI-TR, U7 CP2102N-A02-GQFN28, U8 FPC-SMD_8P-P0.5, U9 FPC-SMD_8P-P0.5

Commit message: update
Parts:
- removed J1: Conn_01x02_Male, Connector_PinHeader_2.54mm:PinHeader_1x02_P2.54mm_Vertical, symbol Connector:Conn_01x02_Male
Changed lines of the file:
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@@
   (junction (at 172.212 39.878) (diameter 0) (color 0 0 0 0)
   )
-  (junction (at 195.072 57.15) (diameter 0) (color 0 0 0 0)
-  )
   (junction (at 535.178 279.908) (diameter 0) (color 0 0 0 0)
   )
@@
   (junction (at 69.342 59.436) (diameter 0) (color 0 0 0 0)
   )
-  (junction (at 210.82 42.672) (diameter 0) (color 0 0 0 0)
-  )
   (junction (at 118.618 159.004) (diameter 0) (color 0 0 0 0)
   )
@@
     (stroke (width 0) (type default) (color 0 0 0 0))
   )
-  (wire (pts (xy 210.82 42.672) (xy 220.472 42.672))
-    (stroke (width 0) (type default) (color 0 0 0 0))
-  )
   (wire (pts (xy 522.478 291.338) (xy 522.478 295.148))
     (stroke (width 0) (type default) (color 0 0 0 0))
@@
     (stroke (width 0) (type default) (color 0 0 0 0))
   )
-  (wire (pts (xy 195.072 57.15) (xy 195.072 61.722))
-    (stroke (width 0) (type default) (color 0 0 0 0))
-  )
   (wire (pts (xy 346.71 222.25) (xy 346.71 234.95))
     (stroke (width 0) (type default) (color 0 0 0 0))
@@
     (stroke (width 0) (type default) (color 0 0 0 0))
   )
-  (wire (pts (xy 202.692 42.672) (xy 210.82 42.672))
+  (wire (pts (xy 202.692 42.672) (xy 220.472 42.672))
     (stroke (width 0) (type default) (color 0 0 0 0))
   )
@@
     (stroke (width 0) (type default) (color 0 0 0 0))
   )
-  (wire (pts (xy 195.072 50.292) (xy 195.072 57.15))
+  (wire (pts (xy 195.072 50.292) (xy 195.072 61.722))
     (stroke (width 0) (type default) (color 0 0 0 0))
   )
@@
     (stroke (width 0) (type default) (color 0 0 0 0))
   )
-  (wire (pts (xy 208.28 71.374) (xy 208.28 57.15))
-    (stroke (width 0) (type default) (color 0 0 0 0))
-  )
   (polyline (pts (xy 273.812 292.608) (xy 273.812 399.542))
     (stroke (width 0) (type default) (color 0 0 0 0))
@@
     (stroke (width 0) (type default) (color 0 0 0 0))
   )
-  (wire (pts (xy 208.28 57.15) (xy 195.072 57.15))
-    (stroke (width 0) (type default) (color 0 0 0 0))
-  )
   (polyline (pts (xy 443.738 102.616) (xy 443.738 103.886))
     (stroke (width 0) (type default) (color 0 0 0 0))
@@
     (stroke (width 0) (type default) (color 0 0 0 0))
   )
-  (wire (pts (xy 210.82 71.374) (xy 210.82 42.672))
-    (stroke (width 0) (type default) (color 0 0 0 0))
-  )
   (text "USB与串口" (at 389.89 274.32 0)
     (effects (font (size 4.572 4.572)) (justify left bottom))
@@
     (effects (font (size 1.27 1.27)) (justify left bottom))
   )
-  (label "IO33" (at 178.054 315.976 180)
-    (effects (font (size 1.27 1.27)) (justify right bottom))
+  (label "IO33" (at 178.054 315.976 0)
+    (effects (font (size 1.27 1.27)) (justify left bottom))
   )
   (label "IO13" (at 296.926 237.49 180)
@@
     (pin "2")
   )
-  (symbol (lib_id "Connector:Conn_01x02_Male") (at 208.28 76.454 90) (unit 1)
-    (in_bom yes) (on_board yes)
-    (property "Reference" "J1" (id 0) (at 211.836 74.5489 90)
-      (effects (font (size 1.27 1.27)) (justify right))
-    )
-    (property "Value" "Conn_01x02_Male" (id 1) (at 201.676 78.994 90)
-      (effects (font (size 1.27 1.27)) (justify right))
-    )
-    (property "Footprint" "Connector_PinHeader_2.54mm:PinHeader_1x02_P2.54mm_Vertical" (id 2) (at 208.28 76.454 0)
-      (effects (font (size 1.27 1.27)) hide)
-    )
-    (property "Datasheet" "~" (id 3) (at 208.28 76.454 0)
-      (effects (font (size 1.27 1.27)) hide)
-    )
-    (pin "1")
-    (pin "2")
-  )
   (symbol (lib_id "Device:C") (at 172.212 54.102 0) (unit 1)
     (in_bom yes) (on_board yes) (fields_autoplaced)
@@
       (reference "D1") (unit 1) (value "Red LED") (footprint "LED_SMD:LED_0603_1608Metric")
     )
-    (path "/d96f9893-c62f-4f43-b5ae-b0c08e7930fa"
-      (reference "J1") (unit 1) (value "Conn_01x02_Male") (footprint "Connector_PinHeader_2.54mm:PinHeader_1x02_P2.54mm_Vertical")
-    )
     (path "/14e49118-6fa6-4ece-a73c-9c09531f18da"

Commit message: update
Connections:
- net GND: now also Card1.6 (VSS), Card1.9 (CD); no longer Card1.1 (DAT2), Card1.4 (VDD)
- net IO13: now also Card1.3 (CMD); no longer Card1.7 (DAT0)
- net IO15: now also Card1.2 (CD/DAT3); no longer Card1.8 (DAT1)
- net IO26: now also Card1.7 (DAT0); no longer Card1.3 (CMD)
- net VDD33: now also Card1.4 (VDD); no longer Card1.6 (VSS)
